File: VCU_V3.3/APPS.kicad_sch (KiCad schematic)
At the start: 6 parts, among them U6 OP07

Commit message: funny stuffs
Parts:
- R24, R25: value R -> 680R
Changed lines of the file:
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@@
 			)
 		)
-		(property "Value" "R"
+		(property "Value" "680R"
 			(at 109.22 96.5199 0)
 			(effects
@@
 			)
 		)
-		(property "Value" "R"
+		(property "Value" "680R"
 			(at 109.22 78.7399 0)
 			(effects
