File: VCU_V3.3/APPS_gain.kicad_sch (KiCad schematic)
At the start: 8 parts, among them U7 OP07

Commit message: funny stuffs
Parts:
- R26: value R -> 2k
- R27: value R -> 330R
Changed lines of the file:
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@@
 			)
 		)
-		(property "Value" "R"
+		(property "Value" "330R"
 			(at 92.71 96.5199 0)
 			(effects
@@
 			)
 		)
-		(property "Value" "R"
+		(property "Value" "2k"
 			(at 92.71 78.7399 0)
 			(effects
