File: VCU_V3.3/AIN.kicad_sch (KiCad schematic)
At the start: 6 parts, among them U13 SGM722

Commit message: VCU3.3 UPDATES
Parts:
- renumbered C30 to C51, C31 to C52, C38 to C53, C37 to C54, C32 to C55, U13 to U16
