File: VCU_V3.3/PDU_P4.kicad_sch (KiCad schematic)
At the start: 9 parts, among them U12 LTV-847S

Commit message: VCU3.3 UPDATES
Parts:
- U12: footprint to be sorted:SMDIP-16_W9.53mm -> RMC_SO:SOIC-16_3.9x9.9mm_P1.27mm_Handsolder
