File: VCU_V3.3/LM2575 AMS1117.kicad_sch (KiCad schematic)
At the start: 10 parts, among them U2 LM2575-5.0BU

Commit message: VCU3.3 UPDATES
Parts:
- removed C10, C15: 100nF, RMC_Capacitor:C_0805_2012Metric_Pad1.18x1.45mm_HandSolder_L, symbol Device:C
- removed C14: 330uF, RMC_Capacitor:CP_Radial_D6.3mm_P2.50mm_handsolder, symbol Device:C_Polarized
- removed C8: 100uF, RMC_Capacitor:CP_Radial_D6.3mm_P2.50mm_handsolder, symbol Device:C_Polarized
- removed D1: SS32, Diode_SMD:D_SMA_Handsoldering, symbol Device:D_Schottky
- removed D9: LED, RMC_LED:LED_0805_2012Metric_Pad1.45x1.40mm_HandSolder, symbol Device:LED
- removed F1: 12V 3A, Fuse:Fuse_1210_3225Metric_Pad1.42x2.65mm_HandSolder, symbol Device:Fuse
- removed L1: 330uH, RMC_Inductor:L_TDK_SLF12575, symbol Device:L
- removed R69: 1k, RMC_Resistor:R_0805_2012Metric_Pad1.20x1.40mm_HandSolder_L, symbol Device:R
- removed U2: LM2575-5.0BU, RMC_TO:TO-263-5_TabPin3_Long, symbol Regulator_Switching:LM2575-5.0BU
- added C40: 47uF, RMC_Capacitor:C_1210_3225Metric_Pad1.33x2.70mm_HandSolder, symbol Device:C_Polarized
- added C42: 10uF, RMC_Capacitor:C_0805_2012Metric_Pad1.18x1.45mm_HandSolder_L, symbol Device:C_Polarized
- added C45, C47, C50: 100nF, RMC_Capacitor:C_0805_2012Metric_Pad1.18x1.45mm_HandSolder_L, symbol Device:C
- added C48, C49: 22uF, RMC_Capacitor:C_0805_2012Metric_Pad1.18x1.45mm_HandSolder_L, symbol Device:C_Polarized
- added F3: Fuse, to be sorted:Fuse_1210_3225Metric_Pad1.42x2.65mm_HandSolder, symbol Device:Fuse
- added L2: 10uH, Inductor_SMD:L_6.3x6.3_H3, symbol Device:L
- added R80: 49R9, RMC_Resistor:R_0805_2012Metric_Pad1.20x1.40mm_HandSolder_L, symbol Device:R
- added R81: 100k, RMC_Resistor:R_0805_2012Metric_Pad1.20x1.40mm_HandSolder_L, symbol Device:R
- added R82: 13k3, RMC_Resistor:R_0805_2012Metric_Pad1.20x1.40mm_HandSolder_L, symbol Device:R
- added U18: TPS54302, RMC_SOT:SOT-23-6_Handsoldering_Extended_RMC, symbol Regulator_Switching:TPS54302
Connections:
- net +12V: now also C40.1, C42.1, C45.2, U18.3 (VIN)
- net +5V: now also F3.2
- net GND: now also C40.2, C42.2, C45.1, C48.2, C49.2, C50.1, R82.2, U18.1 (GND)
- new net: R80.2, R81.1
- new net: R81.2, R82.1, U18.4 (FB)
- new net: C47.2, L2.1, U18.2 (SW)
- new net: C47.1, U18.6 (BOOT)
- new net vout: C48.1, C49.1, C50.2, F3.1, L2.2, R80.1
- no-connect marks 0 -> 1
Other:
- note added: "5 = 0.596 * [R2/R3 + 1]"
