File: VCU_V3.3/MCP2515+ TJA1051.kicad_sch (KiCad schematic)
At the start: 10 parts, among them U4 MCP2515-xST, U5 TJA1051T, Y2 20MHz

Commit message: VCU3.3 UPDATES
Connections:
- net INT: now reaches U4.13 (~{INT})
- net XTAL1: no longer names the net of C17.1, R21.1, U4.9 (OSC1), Y2.2
- net XTAL2: no longer names the net of C16.1, R21.2, U4.8 (OSC2), Y2.1
- no-connect marks 7 -> 6

Commit message: edited VCU and  charger
Parts:
- added R83: 47k, RMC_Resistor:R_0805_2012Metric_Pad1.20x1.40mm_HandSolder_L, symbol Device:R
Connections:
- net +5V: now also R83.1
- net CS: now also R83.2
Changed lines of the file:
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@@
+	)
+	(junction
+		(at 71.12 68.58)
+		(diameter 0)
+		(color 0 0 0 0)
 	)
 	(junction
@@
 	(wire
 		(pts
+			(xy 67.31 68.58) (xy 71.12 68.58)
+		)
+		(stroke
+			(width 0)
+			(type default)
+		)
+	)
+	(wire
+		(pts
 			(xy 91.44 83.82) (xy 69.85 83.82)
 		)
@@
 		(pts
 			(xy 121.92 63.5) (xy 129.54 63.5)
+		)
+		(stroke
+			(width 0)
+			(type default)
+		)
+	)
+	(wire
+		(pts
+			(xy 71.12 68.58) (xy 91.44 68.58)
 		)
 		(stroke
@@
 	(hierarchical_label "CS"
 		(shape input)
-		(at 91.44 68.58 180)
+		(at 67.31 68.58 180)
 		(effects
 			(font
@@
 	)
 	(symbol
+		(lib_id "Device:R")
+		(at 71.12 64.77 0)
+		(unit 1)
+		(body_style 1)
+		(exclude_from_sim no)
+		(in_bom yes)
+		(on_board yes)
+		(in_pos_files yes)
+		(dnp no)
+		(fields_autoplaced yes)
+		(property "Reference" "R83"
+			(at 73.66 63.4999 0)
+			(show_name no)
+			(do_not_autoplace no)
+			(effects
+				(font
+					(size 1.27 1.27)
+				)
+				(justify left)
+			)
+		)
+		(property "Value" "47k"
+			(at 73.66 66.0399 0)
+			(show_name no)
+			(do_not_autoplace no)
+			(effects
+				(font
+					(size 1.27 1.27)
+				)
+				(justify left)
+			)
+		)
+		(property "Footprint" "RMC_Resistor:R_0805_2012Metric_Pad1.20x1.40mm_HandSolder_L"
+			(at 69.342 64.77 90)
+			(hide yes)
+			(show_name no)
+			(do_not_autoplace no)
+			(effects
+				(font
+					(size 1.27 1.27)
+				)
+			)
+		)
+		(property "Datasheet" ""
+			(at 71.12 64.77 0)
+			(hide yes)
+			(show_name no)
+			(do_not_autoplace no)
+			(effects
+				(font
+					(size 1.27 1.27)
+				)
+			)
+		)
+		(property "Description" "Resistor"
+			(at 71.12 64.77 0)
+			(hide yes)
+			(show_name no)
+			(do_not_autoplace no)
+			(effects
+				(font
+					(size 1.27 1.27)
+				)
+			)
+		)
+		(pin "1"
+		)
+		(pin "2"
+		)
+		(instances
+			(project "VCU_V3.3"
+				(path "/763833dc-bbcb-46fa-abab-1e60581348ee/8122f23e-c381-4ae5-b34a-5abe261e4548"
+					(reference "R84")
+					(unit 1)
+				)
+				(path "/763833dc-bbcb-46fa-abab-1e60581348ee/baac5f27-d3eb-4504-9f83-90b722b437aa"
+					(reference "R85")
+					(unit 1)
+				)
+				(path "/763833dc-bbcb-46fa-abab-1e60581348ee/d99a1d8c-b439-4a46-9d7e-503c303d1fb2"
+					(reference "R83")
+					(unit 1)
+				)
+			)
+		)
+	)
+	(symbol
 		(lib_id "power:GND")
 		(at 137.16 76.2 0)
@@
 					(unit 1)
 				)
+			)
+		)
+	)
+	(symbol
+		(lib_id "power:+5V")
+		(at 71.12 60.96 0)
+		(unit 1)
+		(body_style 1)
+		(exclude_from_sim no)
+		(in_bom yes)
+		(on_board yes)
+		(in_pos_files yes)
+		(dnp no)
+		(fields_autoplaced yes)
+		(property "Reference" "#PWR053"
+			(at 71.12 64.77 0)
+			(hide yes)
+			(show_name no)
+			(do_not_autoplace no)
+			(effects
+				(font
+					(size 1.27 1.27)
+				)
+			)
+		)
+		(property "Value" "+5V"
+			(at 71.12 55.88 0)
+			(show_name no)
+			(do_not_autoplace no)
+			(effects
+				(font
+					(size 1.27 1.27)
+				)
+			)
+		)
+		(property "Footprint" ""
+			(at 71.12 60.96 0)
+			(hide yes)
+			(show_name no)
+			(do_not_autoplace no)
+			(effects
+				(font
+					(size 1.27 1.27)
+				)
+			)
+		)
+		(property "Datasheet" ""
+			(at 71.12 60.96 0)
+			(hide yes)
+			(show_name no)
+			(do_not_autoplace no)
+			(effects
+				(font
+					(size 1.27 1.27)
+				)
+			)
+		)
+		(property "Description" "Power symbol creates a global label with name \"+5V\""
+			(at 71.12 60.96 0)
+			(hide yes)
+			(show_name no)
+			(do_not_autoplace no)
+			(effects
+				(font
+					(size 1.27 1.27)
+				)
+			)
+		)
+		(pin "1"
+		)
+		(instances
+			(project "VCU_V3.3"
+				(path "/763833dc-bbcb-46fa-abab-1e60581348ee/8122f23e-c381-4ae5-b34a-5abe261e4548"
+					(reference "#PWR054")
+					(unit 1)
+				)
+				(path "/763833dc-bbcb-46fa-abab-1e60581348ee/baac5f27-d3eb-4504-9f83-90b722b437aa"
+					(reference "#PWR055")
+					(unit 1)
+				)
+				(path "/763833dc-bbcb-46fa-abab-1e60581348ee/d99a1d8c-b439-4a46-9d7e-503c303d1fb2"
+					(reference "#PWR053")
+					(unit 1)
+				)
