File: VCU_V3.3/VCU_V3.3.kicad_pcb (KiCad board)
At the start: 2 copper layers, 114 x 95 mm, 150 parts, among them J3 AVR-ISP-6, Q1 MMBT3904, Q2 BSC030P03NS3, Q3 MMBT3904, Q4 BSC030P03NS3, Q5 MMBT3904, Q6 BSC030P03NS3, Q7 MMBT3904, Q8 BSC030P03NS3, SW1 SW_Push, U1 ATmega328P-A, U10 40106, U11 ELQ3H7, U12 LTV-847S, U13 SGM722, U14 MCP2515-xST, U15 TJA1051T, U16 SGM722, U17 SGM722, U18 TPS54302, U4 MCP2515-xST, U5 TJA1051T, U8 MCP2515-xST, U9 TJA1051T, Y1 16MHz, Y2 20MHz, Y3 20MHz, Y4 20MHz

Commit message: shit board
Parts:
- moved R77 15.1 mm to (95.8, 88.1)
- moved R75 6.90 mm to (98.5, 88.1)
- moved J3 2.83 mm to (181.5, 48.5)
- moved C35 2.25 mm to (198.3, 115.5)
- moved R76 1.84 mm to (111.8, 88.1)
- moved C36 1.55 mm to (198.3, 118.7)
- moved R70 1.21 mm to (109.1, 88.1)
- moved R41 1.08 mm to (166.9, 87.2)
- moved R72 1.02 mm to (199.9, 121.8)
- moved R45 0.92 mm to (181.9, 87.2)
- moved R85 0.84 mm to (199.9, 124.1)
- moved R44 0.58 mm to (166.9, 94.8)
- moved R42 0.56 mm to (166.9, 89.7)
- moved R46 0.50 mm to (181.9, 89.7)
- moved R48 0.46 mm to (181.9, 94.8)
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Routing:
- net SCK: track 0.00 -> 161.4 mm, vias 0 -> 2
- net MOSI: track 0.00 -> 121.7 mm, vias 0 -> 2
- net MISO: track 0.00 -> 103.1 mm, vias 0 -> 3
- net +5V: track 90.6 -> 193.2 mm, vias 0 -> 2
- net CS_Debug_CAN: track 4.33 -> 65.5 mm, vias 0 -> 2
- net RESET: track 0.00 -> 55.1 mm
- net OUT_4: track 2.19 -> 49.6 mm, vias 0 -> 1
- net APPS_5VOUT: track 0.00 -> 30.1 mm, vias 0 -> 1
- net DIN5V_4: track 3.54 -> 29.5 mm, vias 0 -> 2
- net CURRENT_LO: track 4.09 -> 29.0 mm
- net DIN5V_1: track 3.43 -> 28.3 mm, vias 0 -> 2
- net DIN5V_3: track 3.34 -> 26.6 mm, vias 0 -> 2
- net APPS_3VOUT: track 0.00 -> 21.9 mm
- net +12V: track 133.7 -> 154.7 mm
- net APPS_3VIN: track 0.00 -> 20.0 mm, vias 0 -> 1
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
Commit message: helo
Parts:
- moved C18 2.34 mm to (173.5, 115.5)
- moved C28 2.16 mm to (149.5, 115.5)
- moved C19 1.67 mm to (173.5, 118.7)
- moved R31 1.61 mm to (151.5, 121.8)
- moved R84 1.53 mm to (151.5, 124.1)
- moved C29 1.40 mm to (149.5, 118.7)
- moved R22 1.09 mm to (175.5, 121.9)
- moved R83 0.99 mm to (175.5, 124.1)
- moved R85 0.61 mm to (200.5, 124.1)
- moved R72 0.61 mm to (200.5, 121.8)
Routing:
- net AMS_INT: track 0.00 -> 96.9 mm, vias 0 -> 2
- net Motor_INT: track 0.00 -> 91.3 mm, vias 0 -> 1
- net CS_Motor_CAN: track 4.33 -> 84.6 mm, vias 0 -> 2
- net MISO: track 103.1 -> 174.3 mm
- net Debug_INT: track 0.00 -> 63.3 mm, vias 0 -> 2
- net CS_AMS_CAN: track 4.33 -> 59.8 mm, vias 0 -> 2
- net MOSI: track 121.7 -> 167.8 mm
- net SCK: track 161.4 -> 169.2 mm, vias 2 -> 3
- net GND: track 4.81 -> 0.00 mm, vias 0 -> 1
- net Net-(U8-~{RESET}): track 3.16 -> 4.45 mm
- net +5V: track 193.2 -> 192.2 mm

Commit message: vcu update not complete
Parts:
- moved R73 81.4 mm to (113.4, 127.6), turned to -90 degrees
- moved G*** 76.8 mm to (263.6, 78.4)
- moved R23 56.4 mm to (113.4, 122.9), turned to 90 degrees
- moved R32 31.6 mm to (113.4, 118.2), turned to 90 degrees
- moved C44 2.80 mm to (134.2, 95.1)
- moved C43 2.80 mm to (134.2, 89.7)
- moved C46 2.80 mm to (134.2, 92.4)
- moved C39 2.80 mm to (117.7, 95.8)
- moved C41 2.80 mm to (117.7, 88.9)
- moved R78 2.80 mm to (117.8, 93.5)
- moved R79 2.80 mm to (117.8, 91.2)
- moved U17 2.80 mm to (125.8, 94.0)
- moved C31 2.70 mm to (134.0, 104.3)
- moved C37 2.70 mm to (134.0, 101.8)
- moved C30 2.70 mm to (117.4, 102.9)
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Routing:
- net +5V: track 192.2 -> 432.9 mm, vias 2 -> 3
- net CAN3-: track 4.19 -> 118.0 mm, vias 0 -> 2
- net CAN3+: track 4.18 -> 118.0 mm, vias 0 -> 2
- net APPS_3V3: track 6.53 -> 110.2 mm, vias 0 -> 2
- net BRAKE_AIN_MCU: track 9.32 -> 104.6 mm, vias 0 -> 2
- net CURRENT_HI_MCU: track 9.32 -> 104.6 mm, vias 0 -> 2
- net APPS_5V: track 10.2 -> 98.4 mm, vias 0 -> 2
- net CURRENT_LO_MCU: track 9.89 -> 94.0 mm, vias 0 -> 2
- net CAN2+: track 4.18 -> 72.4 mm, vias 0 -> 2
- net CAN2-: track 4.18 -> 71.9 mm, vias 0 -> 2
- net RESET: track 55.1 -> 102.6 mm, vias 0 -> 1
- net CAN1-: track 4.18 -> 41.1 mm
- net CAN1+: track 4.18 -> 38.6 mm
- net +12V: track 154.7 -> 167.6 mm
- net APPS_3VOUT: track 21.9 -> 29.2 mm, vias 0 -> 1
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Other:
- board text added: "RBR_VCU_V3.4 08/29/2026 PCB by Nicholas Chan Code by Carson Cheung"
- board text removed: "RBR_VCU_V3.4 08/09/2026 PCB by Nicholas Chan Code by Carson Cheung"

Commit message: update silkscreen
Parts:
- moved G*** 88.4 mm to (175.2, 77.5)

Commit message: final update for 3.4 I think
Parts:
- J1: footprint Better_Handsolder:HD241_GF30 -> RMC_Connnector:HD241_GF30
Connections:
- J1 pad 15: unconnected-(J1-Pad15) -> GND
- J1 pad 23: unconnected-(J1-Pad23) -> GND
- J1 pad 7: unconnected-(J1-Pad7) -> GND
Routing:
- net CAN2-: track 71.9 -> 71.3 mm
Other:
- board text added: "A5G A3G GND GND GND C3H C3L GND"
- board text added: "A5O A3O BRK CURH CURL C2H C2L GND"
- board text added: "AP5I AP3I 5V 5V 5V C1H C1L GND"
- board text added: "D1 D2 D3 D4"
- board text removed: "5V P5 P6 P7"
- board text removed: "A5G A3G GND GND D1 D2 D3 D4"
- board text removed: "A5O A3O BRK CUR CAN3L CAN3H CAN2L CAN2H"
- board text removed: "AP5I AP3I 5V 5V CAN1L CAN1H CAN2L CAN2H"
