File: Charger/untitled.kicad_sch (KiCad schematic)
At the start: 8 parts, among them U5 74LVC1G17, U6 LTV-817S

Commit message: Charger WIP
Parts:
- renumbered U6 to U, U5 to U
Connections:
- net INPUT renamed IN
Changed lines of the file:
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@@
 	)
 	(hierarchical_label "OUT"
-		(shape input)
+		(shape output)
 		(at 134.62 33.02 0)
 		(effects
@@
 		)
 	)
-	(hierarchical_label "INPUT"
+	(hierarchical_label "IN"
 		(shape input)
 		(at 29.21 33.02 180)
@@
 					(unit 1)
 				)
+				(path "/ba218c5d-b6ee-4635-9cf5-de406e83bbdf/94b4f82c-a5cd-441e-ad50-373ea9761a70"
+					(reference "#PWR050")
+					(unit 1)
+				)
+				(path "/ba218c5d-b6ee-4635-9cf5-de406e83bbdf/b4005320-c05e-4a0a-914e-9c80de761f26"
+					(reference "#PWR056")
+					(unit 1)
+				)
 			)
 		)
@@
 					(unit 1)
 				)
+				(path "/ba218c5d-b6ee-4635-9cf5-de406e83bbdf/94b4f82c-a5cd-441e-ad50-373ea9761a70"
+					(reference "CA2")
+					(unit 1)
+				)
+				(path "/ba218c5d-b6ee-4635-9cf5-de406e83bbdf/b4005320-c05e-4a0a-914e-9c80de761f26"
+					(reference "CA3")
+					(unit 1)
+				)
 			)
 		)
@@
 					(unit 1)
 				)
+				(path "/ba218c5d-b6ee-4635-9cf5-de406e83bbdf/94b4f82c-a5cd-441e-ad50-373ea9761a70"
+					(reference "R23")
+					(unit 1)
+				)
+				(path "/ba218c5d-b6ee-4635-9cf5-de406e83bbdf/b4005320-c05e-4a0a-914e-9c80de761f26"
+					(reference "R31")
+					(unit 1)
+				)
 			)
 		)
@@
 					(unit 1)
 				)
+				(path "/ba218c5d-b6ee-4635-9cf5-de406e83bbdf/94b4f82c-a5cd-441e-ad50-373ea9761a70"
+					(reference "R21")
+					(unit 1)
+				)
+				(path "/ba218c5d-b6ee-4635-9cf5-de406e83bbdf/b4005320-c05e-4a0a-914e-9c80de761f26"
+					(reference "R29")
+					(unit 1)
+				)
 			)
 		)
@@
 					(unit 1)
 				)
+				(path "/ba218c5d-b6ee-4635-9cf5-de406e83bbdf/94b4f82c-a5cd-441e-ad50-373ea9761a70"
+					(reference "R22")
+					(unit 1)
+				)
+				(path "/ba218c5d-b6ee-4635-9cf5-de406e83bbdf/b4005320-c05e-4a0a-914e-9c80de761f26"
+					(reference "R30")
+					(unit 1)
+				)
 			)
 		)
@@
 		(dnp no)
 		(fields_autoplaced yes)
-		(property "Reference" "U6"
+		(property "Reference" "U"
 			(at 116.84 26.67 0)
 			(effects
@@
 		)
 		(instances
-			(project ""
-				(path "/ba218c5d-b6ee-4635-9cf5-de406e83bbdf/555d9f29-2dec-4b3b-ab31-34f0714418de"
-					(reference "U6")
+			(project "Charger"
+				(path "/ba218c5d-b6ee-4635-9cf5-de406e83bbdf/94b4f82c-a5cd-441e-ad50-373ea9761a70"
+					(reference "U9")
+					(unit 1)
+				)
+				(path "/ba218c5d-b6ee-4635-9cf5-de406e83bbdf/b4005320-c05e-4a0a-914e-9c80de761f26"
+					(reference "U11")
 					(unit 1)
 				)
@@
 					(unit 1)
 				)
+				(path "/ba218c5d-b6ee-4635-9cf5-de406e83bbdf/94b4f82c-a5cd-441e-ad50-373ea9761a70"
+					(reference "#PWR047")
+					(unit 1)
+				)
+				(path "/ba218c5d-b6ee-4635-9cf5-de406e83bbdf/b4005320-c05e-4a0a-914e-9c80de761f26"
+					(reference "#PWR053")
+					(unit 1)
+				)
 			)
 		)
@@
 					(unit 1)
 				)
+				(path "/ba218c5d-b6ee-4635-9cf5-de406e83bbdf/94b4f82c-a5cd-441e-ad50-373ea9761a70"
+					(reference "#PWR048")
+					(unit 1)
+				)
+				(path "/ba218c5d-b6ee-4635-9cf5-de406e83bbdf/b4005320-c05e-4a0a-914e-9c80de761f26"
+					(reference "#PWR054")
+					(unit 1)
+				)
 			)
 		)
@@
 					(unit 1)
 				)
+				(path "/ba218c5d-b6ee-4635-9cf5-de406e83bbdf/94b4f82c-a5cd-441e-ad50-373ea9761a70"
+					(reference "#PWR051")
+					(unit 1)
+				)
+				(path "/ba218c5d-b6ee-4635-9cf5-de406e83bbdf/b4005320-c05e-4a0a-914e-9c80de761f26"
+					(reference "#PWR057")
+					(unit 1)
+				)
 			)
 		)
@@
 					(unit 1)
 				)
+				(path "/ba218c5d-b6ee-4635-9cf5-de406e83bbdf/94b4f82c-a5cd-441e-ad50-373ea9761a70"
+					(reference "R20")
+					(unit 1)
+				)
+				(path "/ba218c5d-b6ee-4635-9cf5-de406e83bbdf/b4005320-c05e-4a0a-914e-9c80de761f26"
+					(reference "R24")
+					(unit 1)
+				)
 			)
 		)
@@
 		(on_board yes)
 		(dnp no)
-		(property "Reference" "U5"
+		(property "Reference" "U"
 			(at 91.694 24.638 0)
 			(effects
@@
 		)
 		(instances
-			(project ""
-				(path "/ba218c5d-b6ee-4635-9cf5-de406e83bbdf/555d9f29-2dec-4b3b-ab31-34f0714418de"
-					(reference "U5")
+			(project "Charger"
+				(path "/ba218c5d-b6ee-4635-9cf5-de406e83bbdf/94b4f82c-a5cd-441e-ad50-373ea9761a70"
+					(reference "U8")
+					(unit 1)
+				)
+				(path "/ba218c5d-b6ee-4635-9cf5-de406e83bbdf/b4005320-c05e-4a0a-914e-9c80de761f26"
+					(reference "U10")
 					(unit 1)
 				)
@@
 					(unit 1)
 				)
+				(path "/ba218c5d-b6ee-4635-9cf5-de406e83bbdf/94b4f82c-a5cd-441e-ad50-373ea9761a70"
+					(reference "#PWR052")
+					(unit 1)
+				)
+				(path "/ba218c5d-b6ee-4635-9cf5-de406e83bbdf/b4005320-c05e-4a0a-914e-9c80de761f26"
+					(reference "#PWR058")
+					(unit 1)
+				)
 			)
 		)
@@
 				(path "/ba218c5d-b6ee-4635-9cf5-de406e83bbdf/555d9f29-2dec-4b3b-ab31-34f0714418de"
 					(reference "#PWR032")
+					(unit 1)
+				)
+				(path "/ba218c5d-b6ee-4635-9cf5-de406e83bbdf/94b4f82c-a5cd-441e-ad50-373ea9761a70"
+					(reference "#PWR049")
+					(unit 1)
+				)
+				(path "/ba218c5d-b6ee-4635-9cf5-de406e83bbdf/b4005320-c05e-4a0a-914e-9c80de761f26"
+					(reference "#PWR055")
 					(unit 1)
 				)
@@
 					(unit 1)
 				)
+				(path "/ba218c5d-b6ee-4635-9cf5-de406e83bbdf/94b4f82c-a5cd-441e-ad50-373ea9761a70"
+					(reference "D4")
+					(unit 1)
+				)
+				(path "/ba218c5d-b6ee-4635-9cf5-de406e83bbdf/b4005320-c05e-4a0a-914e-9c80de761f26"
+					(reference "D6")
+					(unit 1)
+				)
