File: Charger/DIGIPOT.kicad_sch (KiCad schematic)
At the start: 0 parts

Commit message: Charger WIP
Parts:
- added U2: AD5235BRUZ25, AD5235BRUZ25:SOP65P640X120-16N, symbol AD5235BRUZ25:AD5235BRUZ25
Connections:
- new net +5V: U2.12 (VDD), U2.13 (WP*), U2.14 (PR*)
- new net A1: U2.6 (A1)
- new net A2: U2.11 (A2)
- new net B1: U2.8 (B1)
- new net B2: U2.9 (B2)
- new net CS: U2.15 (CS*)
- new net GND: U2.4 (GND), U2.5 (VSS)
- new net MISO: U2.3 (SDO)
- new net MOSI: U2.2 (SDI)
- new net RDY: U2.16 (RDY)
- new net SCK: U2.1 (CLK)
- new net W1: U2.7 (W1)
- new net W2: U2.10 (W2)

Commit message: charger WIP
Parts:
- renumbered U2 to U5
Changed lines of the file:
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@@
 		(dnp no)
 		(fields_autoplaced yes)
-		(property "Reference" "U2"
+		(property "Reference" "U5"
 			(at 171.45 46.99 0)
 			(effects
@@
 			(project ""
 				(path "/ba218c5d-b6ee-4635-9cf5-de406e83bbdf/723d3193-29c3-4d78-8ff0-96894e34a9dd"
-					(reference "U2")
+					(reference "U5")
 					(unit 1)
 				)
@@
 		(dnp no)
 		(fields_autoplaced yes)
-		(property "Reference" "#PWR019"
+		(property "Reference" "#PWR051"
 			(at 147.32 97.79 0)
 			(effects
@@
 			(project ""
 				(path "/ba218c5d-b6ee-4635-9cf5-de406e83bbdf/723d3193-29c3-4d78-8ff0-96894e34a9dd"
-					(reference "#PWR019")
+					(reference "#PWR051")
 					(unit 1)
 				)
@@
 		(dnp no)
 		(fields_autoplaced yes)
-		(property "Reference" "#PWR018"
+		(property "Reference" "#PWR050"
 			(at 140.97 63.5 0)
 			(effects
@@
 			(project ""
 				(path "/ba218c5d-b6ee-4635-9cf5-de406e83bbdf/723d3193-29c3-4d78-8ff0-96894e34a9dd"
-					(reference "#PWR018")
+					(reference "#PWR050")
 					(unit 1)
 				)
