File: BDUCU/12v_output.kicad_sch (KiCad schematic)
At the start: 0 parts

Commit message: BDUCU did stuffs
Other:
- added sheet POWER_MOS1 (power_mos.kicad_sch)
- added sheet POWER_MOS2 (power_mos.kicad_sch)
- added sheet POWER_MOS3 (power_mos.kicad_sch)

Commit message: bducu updates
Other:
- added sheet POWER_MOS4 (power_mos.kicad_sch)
