File: BDUCU/SDCLATCH.kicad_sch (KiCad schematic)
At the start: 11 parts, among them K1 SANYOU_SRD_Form_C, Q9 AO3401A, U16 4001

Commit message: bducu scheme done, waiting for check
Parts:
- removed K1: SANYOU_SRD_Form_C, Relay_THT:Relay_SPDT_SANYOU_SRD_Series_Form_C, symbol Relay:SANYOU_SRD_Form_C
- added K2: HF49FD-012-1H11T, to be sorted:HF49FD-012-1H11T, symbol Relay:Relay_SPST-NO
- C32: renamed from C33; value 220u -> 220uF
- C33: renamed from C32; value 100n -> 100nF; footprint Capacitor_SMD:C_0805_2012Metric_Pad1.18x1.45mm_HandSolder -> RMC_Capacitor:C_0805_2012Metric_Pad1.18x1.45mm_HandSolder_L
- R52, R69, R70, R71: footprint Resistor_SMD:R_0805_2012Metric_Pad1.20x1.40mm_HandSolder -> RMC_Resistor:R_0805_2012Metric_Pad1.20x1.40mm_HandSolder_L
- R72: renamed from R73; footprint Resistor_SMD:R_0805_2012Metric_Pad1.20x1.40mm_HandSolder -> RMC_Resistor:R_0805_2012Metric_Pad1.20x1.40mm_HandSolder_L
- U16: footprint RMC-KiCad:SOIC127P600X175-14N -> RMC_SO:SOIC127P600X175-14N
Connections:
- net GND: now also K2.A2
- net SDC_IN: now also K2.13
- net SDC_OUT: now also K2.14
- net TSMS_latch: now also U16.3, U16.5; no longer U16.2, U16.4
- net TSMS_relay+: now also K2.A1
- new net: U16.2, U16.4
- no-connect marks 1 -> 0
Other:
- note removed: "NC"

Commit message: Finished BDUCU layout, silkscreen remaining
Parts:
- added C41: 220uF, Capacitor_SMD:C_1210_3225Metric_Pad1.33x2.70mm_HandSolder, symbol Device:C
Connections:
- net +5V: now also C41.1; no longer C32.1
- net TSMS_reset: now also C41.2; no longer C32.2
Other:
- moved on the sheet: C32
Changed lines of the file:
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@@
 	(symbol
 		(lib_id "Device:C_Polarized")
-		(at 55.88 100.33 0)
-		(unit 1)
-		(exclude_from_sim no)
-		(in_bom yes)
-		(on_board yes)
+		(at 72.39 113.03 0)
+		(unit 1)
+		(exclude_from_sim no)
+		(in_bom yes)
+		(on_board no)
 		(dnp no)
 		(fields_autoplaced yes)
 		(property "Reference" "C32"
-			(at 59.69 98.1709 0)
+			(at 76.2 110.8709 0)
 			(effects
 				(font
@@
 		)
 		(property "Value" "220uF"
-			(at 59.69 100.7109 0)
+			(at 76.2 113.4109 0)
 			(effects
 				(font
@@
 		)
 		(property "Footprint" "Capacitor_THT:CP_Radial_D5.0mm_P2.00mm"
-			(at 56.8452 104.14 0)
+			(at 73.3552 116.84 0)
 			(effects
 				(font
@@
 		)
 		(property "Datasheet" "~"
-			(at 55.88 100.33 0)
+			(at 72.39 113.03 0)
 			(effects
 				(font
@@
 		)
 		(property "Description" "Polarized capacitor"
-			(at 55.88 100.33 0)
+			(at 72.39 113.03 0)
 			(effects
 				(font
@@
 					(unit 1)
 				)
+			)
+		)
+	)
+	(symbol
+		(lib_id "Device:C")
+		(at 55.88 100.33 0)
+		(unit 1)
+		(exclude_from_sim no)
+		(in_bom yes)
+		(on_board yes)
+		(dnp no)
+		(fields_autoplaced yes)
+		(property "Reference" "C41"
+			(at 59.69 99.0599 0)
+			(effects
+				(font
+					(size 1.27 1.27)
+				)
+				(justify left)
+			)
+		)
+		(property "Value" "220uF"
+			(at 59.69 101.5999 0)
+			(effects
+				(font
+					(size 1.27 1.27)
+				)
+				(justify left)
+			)
+		)
+		(property "Footprint" "Capacitor_SMD:C_1210_3225Metric_Pad1.33x2.70mm_HandSolder"
+			(at 56.8452 104.14 0)
+			(effects
+				(font
+					(size 1.27 1.27)
+				)
+				(hide yes)
+			)
+		)
+		(property "Datasheet" "~"
+			(at 55.88 100.33 0)
+			(effects
+				(font
+					(size 1.27 1.27)
+				)
+				(hide yes)
+			)
+		)
+		(property "Description" "Unpolarized capacitor"
+			(at 55.88 100.33 0)
+			(effects
+				(font
+					(size 1.27 1.27)
+				)
+				(hide yes)
+			)
+		)
+		(pin "2"
+		)
+		(pin "1"
+		)
+		(instances
+			(project ""
+				(path "/9942a424-e19d-4ffb-8473-f960b5c811cf/35f5b11b-5d0d-4700-8479-f25bb26aecd1/1890627c-a006-4e49-97ad-50a658112688"
+					(reference "C41")
+					(unit 1)
+				)

Commit message: bomupdates
Parts:
- C32: now left out of the parts list
- C41: Price (none) -> 3.3
- K2: Price (none) -> 3.5
Changed lines of the file:
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@@
 		(unit 1)
 		(exclude_from_sim no)
-		(in_bom yes)
+		(in_bom no)
 		(on_board no)
 		(dnp no)
@@
 				)
 				(hide yes)
+			)
+		)
+		(property "Price" "3.5"
+			(at 210.82 86.36 0)
+			(effects
+				(font
+					(size 1.27 1.27)
+				)
 			)
 		)
@@
 			)
 		)
+		(property "Price" "3.3"
+			(at 55.88 100.33 0)
+			(effects
+				(font
+					(size 1.27 1.27)
+				)
+			)
+		)

Commit message: I am Nicholas Chan (lesbian version)
Parts:
- renumbered C41 to C33, C32 to C34, C33 to C35, K2 to K1, R52 to R68, U16 to U17
Changed lines of the file:
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@@
 		(dnp no)
 		(fields_autoplaced yes)
-		(property "Reference" "U16"
+		(property "Reference" "U17"
 			(at 116.84 130.8099 0)
 			(effects
@@
 			(project "BDUCU"
 				(path "/9942a424-e19d-4ffb-8473-f960b5c811cf/35f5b11b-5d0d-4700-8479-f25bb26aecd1/1890627c-a006-4e49-97ad-50a658112688"
-					(reference "U16")
+					(reference "U17")
 					(unit 5)
 				)
@@
 		(dnp no)
 		(fields_autoplaced yes)
-		(property "Reference" "#PWR088"
+		(property "Reference" "#PWR0116"
 			(at 45.72 97.79 0)
 			(effects
@@
 			(project "BDUCU"
 				(path "/9942a424-e19d-4ffb-8473-f960b5c811cf/35f5b11b-5d0d-4700-8479-f25bb26aecd1/1890627c-a006-4e49-97ad-50a658112688"
-					(reference "#PWR088")
+					(reference "#PWR0116")
 					(unit 1)
 				)
@@
 		(dnp no)
 		(fields_autoplaced yes)
-		(property "Reference" "U16"
+		(property "Reference" "U17"
 			(at 73.66 59.69 0)
 			(effects
@@
 			(project "BDUCU"
 				(path "/9942a424-e19d-4ffb-8473-f960b5c811cf/35f5b11b-5d0d-4700-8479-f25bb26aecd1/1890627c-a006-4e49-97ad-50a658112688"
-					(reference "U16")
+					(reference "U17")
 					(unit 4)
 				)
@@
 		(dnp no)
 		(fields_autoplaced yes)
-		(property "Reference" "C32"
+		(property "Reference" "C34"
 			(at 76.2 110.8709 0)
 			(effects
@@
 			(project "BDUCU"
 				(path "/9942a424-e19d-4ffb-8473-f960b5c811cf/35f5b11b-5d0d-4700-8479-f25bb26aecd1/1890627c-a006-4e49-97ad-50a658112688"
-					(reference "C32")
+					(reference "C34")
 					(unit 1)
 				)
@@
 		(dnp no)
 		(fields_autoplaced yes)
-		(property "Reference" "#PWR0100"
+		(property "Reference" "#PWR0122"
 			(at 162.56 76.2 0)
 			(effects
@@
 			(project "BDUCU"
 				(path "/9942a424-e19d-4ffb-8473-f960b5c811cf/35f5b11b-5d0d-4700-8479-f25bb26aecd1/1890627c-a006-4e49-97ad-50a658112688"
-					(reference "#PWR0100")
+					(reference "#PWR0122")
 					(unit 1)
 				)
@@
 		(dnp no)
 		(fields_autoplaced yes)
-		(property "Reference" "#PWR092"
+		(property "Reference" "#PWR0119"
 			(at 110.49 151.13 0)
 			(effects
@@
 			(project "BDUCU"
 				(path "/9942a424-e19d-4ffb-8473-f960b5c811cf/35f5b11b-5d0d-4700-8479-f25bb26aecd1/1890627c-a006-4e49-97ad-50a658112688"
-					(reference "#PWR092")
+					(reference "#PWR0119")
 					(unit 1)
 				)
@@
 		(dnp no)
 		(fields_autoplaced yes)
-		(property "Reference" "#PWR093"
+		(property "Reference" "#PWR0120"
 			(at 123.19 125.73 0)
 			(effects
@@
 			(project "BDUCU"
 				(path "/9942a424-e19d-4ffb-8473-f960b5c811cf/35f5b11b-5d0d-4700-8479-f25bb26aecd1/1890627c-a006-4e49-97ad-50a658112688"
-					(reference "#PWR093")
+					(reference "#PWR0120")
 					(unit 1)
 				)
@@
 		(dnp no)
 		(fields_autoplaced yes)
-		(property "Reference" "#PWR091"
+		(property "Reference" "#PWR0118"
 			(at 110.49 116.84 0)
 			(effects
@@
 			(project "BDUCU"
 				(path "/9942a424-e19d-4ffb-8473-f960b5c811cf/35f5b11b-5d0d-4700-8479-f25bb26aecd1/1890627c-a006-4e49-97ad-50a658112688"
-					(reference "#PWR091")
+					(reference "#PWR0118")
 					(unit 1)
 				)
@@
 		(dnp no)
 		(fields_autoplaced yes)
-		(property "Reference" "#PWR094"
+		(property "Reference" "#PWR0121"
 			(at 148.59 100.33 0)
 			(effects
@@
 			(project "BDUCU"
 				(path "/9942a424-e19d-4ffb-8473-f960b5c811cf/35f5b11b-5d0d-4700-8479-f25bb26aecd1/1890627c-a006-4e49-97ad-50a658112688"
-					(reference "#PWR094")
+					(reference "#PWR0121")
 					(unit 1)
 				)
@@
 		(dnp no)
 		(fields_autoplaced yes)
-		(property "Reference" "C33"
+		(property "Reference" "C35"
 			(at 119.38 111.76 90)
 			(effects
@@
 			(project "BDUCU"
 				(path "/9942a424-e19d-4ffb-8473-f960b5c811cf/35f5b11b-5d0d-4700-8479-f25bb26aecd1/1890627c-a006-4e49-97ad-50a658112688"
-					(reference "C33")
+					(reference "C35")
 					(unit 1)
 				)
@@
 		(dnp no)
 		(fields_autoplaced yes)
-		(property "Reference" "K2"
+		(property "Reference" "K1"
 			(at 210.82 71.12 90)
 			(effects
@@
 			(project ""
 				(path "/9942a424-e19d-4ffb-8473-f960b5c811cf/35f5b11b-5d0d-4700-8479-f25bb26aecd1/1890627c-a006-4e49-97ad-50a658112688"
-					(reference "K2")
+					(reference "K1")
 					(unit 1)
 				)
@@
 		(dnp no)
 		(fields_autoplaced yes)
-		(property "Reference" "U16"
+		(property "Reference" "U17"
 			(at 93.98 76.2 0)
 			(effects
@@
 			(project "BDUCU"
 				(path "/9942a424-e19d-4ffb-8473-f960b5c811cf/35f5b11b-5d0d-4700-8479-f25bb26aecd1/1890627c-a006-4e49-97ad-50a658112688"
-					(reference "U16")
+					(reference "U17")
 					(unit 2)
 				)
@@
 		(dnp no)
 		(fields_autoplaced yes)
-		(property "Reference" "U16"
+		(property "Reference" "U17"
 			(at 48.26 59.69 0)
 			(effects
@@
 			(project "BDUCU"
 				(path "/9942a424-e19d-4ffb-8473-f960b5c811cf/35f5b11b-5d0d-4700-8479-f25bb26aecd1/1890627c-a006-4e49-97ad-50a658112688"
-					(reference "U16")
+					(reference "U17")
 					(unit 3)
 				)
@@
 		(dnp no)
 		(fields_autoplaced yes)
-		(property "Reference" "#PWR087"
+		(property "Reference" "#PWR0115"
 			(at 26.67 85.09 0)
 			(effects
@@
 			(project "BDUCU"
 				(path "/9942a424-e19d-4ffb-8473-f960b5c811cf/35f5b11b-5d0d-4700-8479-f25bb26aecd1/1890627c-a006-4e49-97ad-50a658112688"
-					(reference "#PWR087")
+					(reference "#PWR0115")
 					(unit 1)
 				)
@@
 		(dnp no)
 		(fields_autoplaced yes)
-		(property "Reference" "#PWR090"
+		(property "Reference" "#PWR0117"
 			(at 45.72 120.65 0)
 			(effects
@@
 			(project "BDUCU"
 				(path "/9942a424-e19d-4ffb-8473-f960b5c811cf/35f5b11b-5d0d-4700-8479-f25bb26aecd1/1890627c-a006-4e49-97ad-50a658112688"
-					(reference "#PWR090")
+					(reference "#PWR0117")
 					(unit 1)
 				)
@@
 		(dnp no)
 		(fields_autoplaced yes)
-		(property "Reference" "C41"
+		(property "Reference" "C33"
 			(at 59.69 99.0599 0)
 			(effects
@@
 			(project ""
 				(path "/9942a424-e19d-4ffb-8473-f960b5c811cf/35f5b11b-5d0d-4700-8479-f25bb26aecd1/1890627c-a006-4e49-97ad-50a658112688"
-					(reference "C41")
+					(reference "C33")
 					(unit 1)
 				)
@@
 		(dnp no)
 		(fields_autoplaced yes)
-		(property "Reference" "R52"
+		(property "Reference" "R68"
 			(at 29.21 73.6599 0)
 			(effects
@@
 			(project "BDUCU"
 				(path "/9942a424-e19d-4ffb-8473-f960b5c811cf/35f5b11b-5d0d-4700-8479-f25bb26aecd1/1890627c-a006-4e49-97ad-50a658112688"
-					(reference "R52")
+					(reference "R68")
 					(unit 1)
 				)
@@
 		(dnp no)
 		(fields_autoplaced yes)
-		(property "Reference" "U16"
+		(property "Reference" "U17"
 			(at 93.98 62.23 0)
 			(effects
@@
 			(project "BDUCU"
 				(path "/9942a424-e19d-4ffb-8473-f960b5c811cf/35f5b11b-5d0d-4700-8479-f25bb26aecd1/1890627c-a006-4e49-97ad-50a658112688"
-					(reference "U16")
+					(reference "U17")
 					(unit 1)
 				)
@@
 		(dnp no)
 		(fields_autoplaced yes)
-		(property "Reference" "#PWR0101"
+		(property "Reference" "#PWR0123"
 			(at 222.25 97.79 0)
 			(effects
@@
 			(project "BDUCU"
 				(path "/9942a424-e19d-4ffb-8473-f960b5c811cf/35f5b11b-5d0d-4700-8479-f25bb26aecd1/1890627c-a006-4e49-97ad-50a658112688"
-					(reference "#PWR0101")
-					(unit 1)
-				)
+					(reference "#PWR0123")
+					(unit 1)
+				)
