File: BDUCU/SDCLATCH.kicad_sch (KiCad schematic)
At the start: 12 parts, among them K1 HF49FD-012-1H11T, Q9 AO3401A, U17 4001

Commit message: update bducu schematics
Parts:
- removed C33: 220uF, Capacitor_SMD:C_1210_3225Metric_Pad1.33x2.70mm_HandSolder, symbol Device:C
- removed C34: 220uF, Capacitor_THT:CP_Radial_D5.0mm_P2.00mm, symbol Device:C_Polarized
- removed C35: 100nF, RMC_Capacitor:C_0805_2012Metric_Pad1.18x1.45mm_HandSolder_L, symbol Device:C
- removed D12: 1N4148, Diode_THT:D_DO-35_SOD27_P7.62mm_Horizontal, symbol Diode:1N4148
- removed K1: HF49FD-012-1H11T, to be sorted:HF49FD-012-1H11T, symbol Relay:Relay_SPST-NO
- removed Q9: AO3401A, Package_TO_SOT_SMD:SOT-23, symbol Transistor_FET:AO3401A
- removed R68: 1M, RMC_Resistor:R_0805_2012Metric_Pad1.20x1.40mm_HandSolder_L, symbol Device:R
- removed R69, R70: 4.7k, RMC_Resistor:R_0805_2012Metric_Pad1.20x1.40mm_HandSolder_L, symbol Device:R
- removed R71: 100R, RMC_Resistor:R_0805_2012Metric_Pad1.20x1.40mm_HandSolder_L, symbol Device:R
- removed R72: 100k, RMC_Resistor:R_0805_2012Metric_Pad1.20x1.40mm_HandSolder_L, symbol Device:R
- removed U17: 4001, RMC_SO:SOIC127P600X175-14N, symbol 4xxx:4001
Other:
- note removed: "12V LVB-> TSMS switch -> TSMS INPUT"
- note removed: "NO"
- note removed: "Reset by power cycle"
- note removed: "latch if input is high"
