File: BDUCU/can_controller.kicad_sch (KiCad schematic)
At the start: 11 parts, among them U10 TJA1050T_CM_118, U11 MCP2515-xST, Y2 20MHz

Commit message: BDUCU did stuffs
Parts:
- C26, C27: value 22pF -> 12pF
Changed lines of the file:
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@@
           (reference "#PWR052") (unit 1)
+        )
+        (path "/9942a424-e19d-4ffb-8473-f960b5c811cf/8fc427df-2d97-44b9-b479-5014f2f05880/e4047b2f-bef8-49d9-83e0-04d733111886"
+          (reference "#PWR063") (unit 1)
         )
       )
@@
           (reference "#PWR053") (unit 1)
         )
+        (path "/9942a424-e19d-4ffb-8473-f960b5c811cf/8fc427df-2d97-44b9-b479-5014f2f05880/e4047b2f-bef8-49d9-83e0-04d733111886"
+          (reference "#PWR061") (unit 1)
+        )
       )
     )
@@
         (path "/9942a424-e19d-4ffb-8473-f960b5c811cf/8fc427df-2d97-44b9-b479-5014f2f05880/146987db-cc4e-40c2-bab5-0abba2715ce3"
           (reference "R26") (unit 1)
+        )
+        (path "/9942a424-e19d-4ffb-8473-f960b5c811cf/8fc427df-2d97-44b9-b479-5014f2f05880/e4047b2f-bef8-49d9-83e0-04d733111886"
+          (reference "R48") (unit 1)
         )
       )
@@
           (reference "U11") (unit 1)
         )
+        (path "/9942a424-e19d-4ffb-8473-f960b5c811cf/8fc427df-2d97-44b9-b479-5014f2f05880/e4047b2f-bef8-49d9-83e0-04d733111886"
+          (reference "U12") (unit 1)
+        )
       )
     )
@@
           (reference "R27") (unit 1)
         )
+        (path "/9942a424-e19d-4ffb-8473-f960b5c811cf/8fc427df-2d97-44b9-b479-5014f2f05880/e4047b2f-bef8-49d9-83e0-04d733111886"
+          (reference "R51") (unit 1)
+        )
       )
     )
@@
       (effects (font (size 1.27 1.27)))
     )
-    (property "Value" "22pF" (at 98.552 122.682 90)
+    (property "Value" "12pF" (at 98.552 122.682 90)
       (effects (font (size 1.27 1.27)))
     )
@@
           (reference "C27") (unit 1)
         )
+        (path "/9942a424-e19d-4ffb-8473-f960b5c811cf/8fc427df-2d97-44b9-b479-5014f2f05880/e4047b2f-bef8-49d9-83e0-04d733111886"
+          (reference "C28") (unit 1)
+        )
       )
     )
@@
           (reference "#PWR049") (unit 1)
         )
+        (path "/9942a424-e19d-4ffb-8473-f960b5c811cf/8fc427df-2d97-44b9-b479-5014f2f05880/e4047b2f-bef8-49d9-83e0-04d733111886"
+          (reference "#PWR059") (unit 1)
+        )
       )
     )
@@
           (reference "C24") (unit 1)
         )
+        (path "/9942a424-e19d-4ffb-8473-f960b5c811cf/8fc427df-2d97-44b9-b479-5014f2f05880/e4047b2f-bef8-49d9-83e0-04d733111886"
+          (reference "C30") (unit 1)
+        )
       )
     )
@@
         (path "/9942a424-e19d-4ffb-8473-f960b5c811cf/8fc427df-2d97-44b9-b479-5014f2f05880/146987db-cc4e-40c2-bab5-0abba2715ce3"
           (reference "C25") (unit 1)
+        )
+        (path "/9942a424-e19d-4ffb-8473-f960b5c811cf/8fc427df-2d97-44b9-b479-5014f2f05880/e4047b2f-bef8-49d9-83e0-04d733111886"
+          (reference "C29") (unit 1)
         )
       )
@@
         (path "/9942a424-e19d-4ffb-8473-f960b5c811cf/8fc427df-2d97-44b9-b479-5014f2f05880/146987db-cc4e-40c2-bab5-0abba2715ce3"
           (reference "Y2") (unit 1)
+        )
+        (path "/9942a424-e19d-4ffb-8473-f960b5c811cf/8fc427df-2d97-44b9-b479-5014f2f05880/e4047b2f-bef8-49d9-83e0-04d733111886"
+          (reference "Y3") (unit 1)
         )
       )
@@
           (reference "#PWR047") (unit 1)
         )
+        (path "/9942a424-e19d-4ffb-8473-f960b5c811cf/8fc427df-2d97-44b9-b479-5014f2f05880/e4047b2f-bef8-49d9-83e0-04d733111886"
+          (reference "#PWR057") (unit 1)
+        )
       )
     )
@@
           (reference "#PWR054") (unit 1)
         )
+        (path "/9942a424-e19d-4ffb-8473-f960b5c811cf/8fc427df-2d97-44b9-b479-5014f2f05880/e4047b2f-bef8-49d9-83e0-04d733111886"
+          (reference "#PWR043") (unit 1)
+        )
       )
     )
@@
           (reference "#PWR050") (unit 1)
         )
+        (path "/9942a424-e19d-4ffb-8473-f960b5c811cf/8fc427df-2d97-44b9-b479-5014f2f05880/e4047b2f-bef8-49d9-83e0-04d733111886"
+          (reference "#PWR056") (unit 1)
+        )
       )
     )
@@
       (effects (font (size 1.27 1.27)))
     )
-    (property "Value" "22pF" (at 98.552 106.172 90)
+    (property "Value" "12pF" (at 98.552 106.172 90)
       (effects (font (size 1.27 1.27)))
     )
@@
           (reference "C26") (unit 1)
         )
+        (path "/9942a424-e19d-4ffb-8473-f960b5c811cf/8fc427df-2d97-44b9-b479-5014f2f05880/e4047b2f-bef8-49d9-83e0-04d733111886"
+          (reference "C19") (unit 1)
+        )
       )
     )
@@
         (path "/9942a424-e19d-4ffb-8473-f960b5c811cf/8fc427df-2d97-44b9-b479-5014f2f05880/146987db-cc4e-40c2-bab5-0abba2715ce3"
           (reference "#PWR051") (unit 1)
+        )
+        (path "/9942a424-e19d-4ffb-8473-f960b5c811cf/8fc427df-2d97-44b9-b479-5014f2f05880/e4047b2f-bef8-49d9-83e0-04d733111886"
+          (reference "#PWR064") (unit 1)
         )
       )
@@
           (reference "#PWR046") (unit 1)
         )
+        (path "/9942a424-e19d-4ffb-8473-f960b5c811cf/8fc427df-2d97-44b9-b479-5014f2f05880/e4047b2f-bef8-49d9-83e0-04d733111886"
+          (reference "#PWR062") (unit 1)
+        )
       )
     )
@@
           (reference "R28") (unit 1)
         )
+        (path "/9942a424-e19d-4ffb-8473-f960b5c811cf/8fc427df-2d97-44b9-b479-5014f2f05880/e4047b2f-bef8-49d9-83e0-04d733111886"
+          (reference "R49") (unit 1)
+        )
       )
     )
@@
         (path "/9942a424-e19d-4ffb-8473-f960b5c811cf/8fc427df-2d97-44b9-b479-5014f2f05880/146987db-cc4e-40c2-bab5-0abba2715ce3"
           (reference "R29") (unit 1)
+        )
+        (path "/9942a424-e19d-4ffb-8473-f960b5c811cf/8fc427df-2d97-44b9-b479-5014f2f05880/e4047b2f-bef8-49d9-83e0-04d733111886"
+          (reference "R50") (unit 1)
         )
       )
@@
           (reference "#PWR055") (unit 1)
         )
+        (path "/9942a424-e19d-4ffb-8473-f960b5c811cf/8fc427df-2d97-44b9-b479-5014f2f05880/e4047b2f-bef8-49d9-83e0-04d733111886"
+          (reference "#PWR058") (unit 1)
+        )
       )
     )
@@
         (path "/9942a424-e19d-4ffb-8473-f960b5c811cf/8fc427df-2d97-44b9-b479-5014f2f05880/146987db-cc4e-40c2-bab5-0abba2715ce3"
           (reference "#PWR048") (unit 1)
+        )
+        (path "/9942a424-e19d-4ffb-8473-f960b5c811cf/8fc427df-2d97-44b9-b479-5014f2f05880/e4047b2f-bef8-49d9-83e0-04d733111886"
+          (reference "#PWR060") (unit 1)
         )
       )
@@
           (reference "U10") (unit 1)
         )
-      )
+        (path "/9942a424-e19d-4ffb-8473-f960b5c811cf/8fc427df-2d97-44b9-b479-5014f2f05880/e4047b2f-bef8-49d9-83e0-04d733111886"
+          (reference "U13") (unit 1)
+        )
+      )

Commit message: bducu scheme done, waiting for check
Parts:
- U10: footprint Package_SO:SOIC-8_3.9x4.9mm_P1.27mm -> RMC_SO:SOIC-8_3.9x4.9mm_P1.27mm_RMC_Handsolder
Changed lines of the file:
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@@
 			)
 		)
-		(property "Footprint" "Package_SO:SOIC-8_3.9x4.9mm_P1.27mm"
+		(property "Footprint" "RMC_SO:SOIC-8_3.9x4.9mm_P1.27mm_RMC_Handsolder"
 			(at 181.356 89.662 0)
 			(effects
@@
 			)
 		)
-		(property "Description" "\n1/1 Transceiver Half CANbus 8-SO\n"
+		(property "Description" "1/1 Transceiver Half CANbus 8-SO"
 			(at 181.356 89.662 0)
 			(effects

Commit message: I am Nicholas Chan (lesbian version)
Parts:
- added R23: 10k, RMC_Resistor:R_0805_2012Metric_Pad1.20x1.40mm_HandSolder_L, symbol Device:R
- renumbered C26 to C18, C27 to C19, C25 to C20, C24 to C21, R28 to R24, R29 to R25, U11 to U10, U10 to U11, Y2 to Y1
Connections:
- net +5V: now also R23.2
- net CS: now also R23.1; no longer R26.1
- net INT: now reaches U10.13 (~{INT})
- net INT: now also R26.1
- no-connect marks 8 -> 7
Other:
- moved on the sheet: C18, C19, C20, C21, R24, R25, R26, U10, U11, Y1
