File: BDUCU/hv_iso_analog.kicad_sch (KiCad schematic)
At the start: 44 parts, among them U1 LM358, U2 LM358, U7 LM358

Commit message: updated values of the Linear Isolator of BDUCU
Parts:
- C8, C9: value 100nF -> 100nF/1%
- R17, R20: value 10k -> 100k
- R18, R19: value 10k -> 100k/1%
- U1, U2: value LM358 -> SGM722
- U3, U4, U5, U6: value ~ -> (none)
Other:
- note added: "1.63V"
- note added: "1.64V"
- note added: "1.68"
- note added: "2.47V"
- note added: "5.32V"

Commit message: BDUCU schematics change
Changed lines of the file:
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@@
 	)
 	(symbol
-		(lib_id "power:GND")
-		(at 217.424 88.392 0)
-		(unit 1)
-		(body_style 1)
-		(exclude_from_sim no)
-		(in_bom yes)
-		(on_board yes)
-		(in_pos_files yes)
-		(dnp no)
-		(fields_autoplaced yes)
-		(property "Reference" "#PWR027"
-			(at 217.424 94.742 0)
-			(hide yes)
-			(show_name no)
-			(do_not_autoplace no)
-			(effects
-				(font
-					(size 1.27 1.27)
-				)
-			)
-		)
-		(property "Value" "GND"
-			(at 217.424 92.964 0)
-			(show_name no)
-			(do_not_autoplace no)
-			(effects
-				(font
-					(size 1.27 1.27)
-				)
-			)
-		)
-		(property "Footprint" ""
-			(at 217.424 88.392 0)
-			(hide yes)
-			(show_name no)
-			(do_not_autoplace no)
-			(effects
-				(font
-					(size 1.27 1.27)
-				)
-			)
-		)
-		(property "Datasheet" ""
-			(at 217.424 88.392 0)
-			(hide yes)
-			(show_name no)
-			(do_not_autoplace no)
-			(effects
-				(font
-					(size 1.27 1.27)
-				)
-			)
-		)
-		(property "Description" ""
-			(at 217.424 88.392 0)
-			(show_name no)
-			(do_not_autoplace no)
-			(effects
-				(font
-					(size 1.27 1.27)
-				)
-			)
-		)
-		(pin "1"
-		)
-		(instances
-			(project "BDUCU"
-				(path "/9942a424-e19d-4ffb-8473-f960b5c811cf/d0210ccf-eb84-46ca-8cbf-aeaae330deeb"
-					(reference "#PWR027")
-					(unit 1)
-				)
-			)
-		)
-	)
-	(symbol
 		(lib_id "Device:R")
 		(at 163.576 68.58 180)
@@
 		)
 		(property "Value" "100k/1%"
-			(at 197.612 68.072 0)
+			(at 197.612 69.342 0)
 			(show_name no)
 			(do_not_autoplace no)
