File: BDUCU/power_mos.kicad_sch (KiCad schematic)
At the start: 10 parts, among them Q1 MMBT3906, Q2 BSC019N04LS

Commit message: bducu scheme done, waiting for check
Parts:
- removed D5: LED, RMC_LED:LED_0805_2012Metric_Pad1.45x1.40mm_HandSolder, symbol Device:LED
- removed F3: Fuse, RMC_Connnector:3 in 1 fuseholder, symbol Device:Fuse
- removed Q2: BSC019N04LS, RMC_SO:Infineon_PG-TDSON-8_6.15x5.15mm, symbol Transistor_FET:BSC061N08NS5
- removed R32: 1k, RMC_Resistor:R_0805_2012Metric_Pad1.20x1.40mm_HandSolder_L, symbol Device:R
- added Q10: AO3400A, RMC_SOT:SOT-23, symbol Transistor_FET:AO3400A
- Q1: footprint Better_Handsolder:SOT-23 -> RMC_SOT:SOT-23
Connections:
- net GND: now also Q10.2 (S)
- net OUT: now also Q10.3 (D)
- net at D4.2 (A), Q1.3 (C), R30.1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: now also Q10.1 (G)
Other:
- moved on the sheet: D4, Q1, R23, R24, R30

Commit message: I am Nicholas Chan (lesbian version)
Parts:
- renumbered Q10 to Q2, R23 to R31, R24 to R32, R30 to R33, R31 to R34
Changed lines of the file:
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@@
 		(on_board yes)
 		(dnp no)
-		(property "Reference" "R24"
+		(property "Reference" "R32"
 			(at 127.381 94.107 0)
 			(effects
@@
 			(project "BDUCU"
 				(path "/9942a424-e19d-4ffb-8473-f960b5c811cf/db59dc7f-5332-44a2-bb52-28901b78a7e3/57d5af05-edab-40f7-aafe-6a2e0130ba84"
-					(reference "R24")
-					(unit 1)
-				)
-				(path "/9942a424-e19d-4ffb-8473-f960b5c811cf/db59dc7f-5332-44a2-bb52-28901b78a7e3/b88b6ec3-afc4-43aa-baa2-21af531f917d"
-					(reference "R34")
-					(unit 1)
-				)
-				(path "/9942a424-e19d-4ffb-8473-f960b5c811cf/db59dc7f-5332-44a2-bb52-28901b78a7e3/cd40e0a1-5e03-48e1-9b54-a7b8526d72ef"
-					(reference "R39")
+					(reference "R32")
+					(unit 1)
+				)
+				(path "/9942a424-e19d-4ffb-8473-f960b5c811cf/db59dc7f-5332-44a2-bb52-28901b78a7e3/b88b6ec3-afc4-43aa-baa2-21af531f917d"
+					(reference "R36")
+					(unit 1)
+				)
+				(path "/9942a424-e19d-4ffb-8473-f960b5c811cf/db59dc7f-5332-44a2-bb52-28901b78a7e3/cd40e0a1-5e03-48e1-9b54-a7b8526d72ef"
+					(reference "R40")
 					(unit 1)
 				)
@@
 		(on_board yes)
 		(dnp no)
-		(property "Reference" "R31"
+		(property "Reference" "R34"
 			(at 136.271 86.233 0)
 			(effects
@@
 			(project "BDUCU"
 				(path "/9942a424-e19d-4ffb-8473-f960b5c811cf/db59dc7f-5332-44a2-bb52-28901b78a7e3/57d5af05-edab-40f7-aafe-6a2e0130ba84"
-					(reference "R31")
-					(unit 1)
-				)
-				(path "/9942a424-e19d-4ffb-8473-f960b5c811cf/db59dc7f-5332-44a2-bb52-28901b78a7e3/b88b6ec3-afc4-43aa-baa2-21af531f917d"
-					(reference "R36")
-					(unit 1)
-				)
-				(path "/9942a424-e19d-4ffb-8473-f960b5c811cf/db59dc7f-5332-44a2-bb52-28901b78a7e3/cd40e0a1-5e03-48e1-9b54-a7b8526d72ef"
-					(reference "R41")
+					(reference "R34")
+					(unit 1)
+				)
+				(path "/9942a424-e19d-4ffb-8473-f960b5c811cf/db59dc7f-5332-44a2-bb52-28901b78a7e3/b88b6ec3-afc4-43aa-baa2-21af531f917d"
+					(reference "R38")
+					(unit 1)
+				)
+				(path "/9942a424-e19d-4ffb-8473-f960b5c811cf/db59dc7f-5332-44a2-bb52-28901b78a7e3/cd40e0a1-5e03-48e1-9b54-a7b8526d72ef"
+					(reference "R42")
 					(unit 1)
 				)
@@
 		(on_board yes)
 		(dnp no)
-		(property "Reference" "R23"
+		(property "Reference" "R31"
 			(at 119.38 74.168 90)
 			(effects
@@
 			(project "BDUCU"
 				(path "/9942a424-e19d-4ffb-8473-f960b5c811cf/db59dc7f-5332-44a2-bb52-28901b78a7e3/57d5af05-edab-40f7-aafe-6a2e0130ba84"
-					(reference "R23")
-					(unit 1)
-				)
-				(path "/9942a424-e19d-4ffb-8473-f960b5c811cf/db59dc7f-5332-44a2-bb52-28901b78a7e3/b88b6ec3-afc4-43aa-baa2-21af531f917d"
-					(reference "R33")
-					(unit 1)
-				)
-				(path "/9942a424-e19d-4ffb-8473-f960b5c811cf/db59dc7f-5332-44a2-bb52-28901b78a7e3/cd40e0a1-5e03-48e1-9b54-a7b8526d72ef"
-					(reference "R38")
+					(reference "R31")
+					(unit 1)
+				)
+				(path "/9942a424-e19d-4ffb-8473-f960b5c811cf/db59dc7f-5332-44a2-bb52-28901b78a7e3/b88b6ec3-afc4-43aa-baa2-21af531f917d"
+					(reference "R35")
+					(unit 1)
+				)
+				(path "/9942a424-e19d-4ffb-8473-f960b5c811cf/db59dc7f-5332-44a2-bb52-28901b78a7e3/cd40e0a1-5e03-48e1-9b54-a7b8526d72ef"
+					(reference "R39")
 					(unit 1)
 				)
@@
 		(on_board yes)
 		(dnp no)
-		(property "Reference" "R30"
+		(property "Reference" "R33"
 			(at 135.636 76.708 0)
 			(effects
@@
 			(project "BDUCU"
 				(path "/9942a424-e19d-4ffb-8473-f960b5c811cf/db59dc7f-5332-44a2-bb52-28901b78a7e3/57d5af05-edab-40f7-aafe-6a2e0130ba84"
-					(reference "R30")
-					(unit 1)
-				)
-				(path "/9942a424-e19d-4ffb-8473-f960b5c811cf/db59dc7f-5332-44a2-bb52-28901b78a7e3/b88b6ec3-afc4-43aa-baa2-21af531f917d"
-					(reference "R35")
-					(unit 1)
-				)
-				(path "/9942a424-e19d-4ffb-8473-f960b5c811cf/db59dc7f-5332-44a2-bb52-28901b78a7e3/cd40e0a1-5e03-48e1-9b54-a7b8526d72ef"
-					(reference "R40")
+					(reference "R33")
+					(unit 1)
+				)
+				(path "/9942a424-e19d-4ffb-8473-f960b5c811cf/db59dc7f-5332-44a2-bb52-28901b78a7e3/b88b6ec3-afc4-43aa-baa2-21af531f917d"
+					(reference "R37")
+					(unit 1)
+				)
+				(path "/9942a424-e19d-4ffb-8473-f960b5c811cf/db59dc7f-5332-44a2-bb52-28901b78a7e3/cd40e0a1-5e03-48e1-9b54-a7b8526d72ef"
+					(reference "R41")
 					(unit 1)
 				)
@@
 				)
 				(path "/9942a424-e19d-4ffb-8473-f960b5c811cf/db59dc7f-5332-44a2-bb52-28901b78a7e3/b88b6ec3-afc4-43aa-baa2-21af531f917d"
+					(reference "D5")
+					(unit 1)
+				)
+				(path "/9942a424-e19d-4ffb-8473-f960b5c811cf/db59dc7f-5332-44a2-bb52-28901b78a7e3/cd40e0a1-5e03-48e1-9b54-a7b8526d72ef"
 					(reference "D6")
 					(unit 1)
 				)
-				(path "/9942a424-e19d-4ffb-8473-f960b5c811cf/db59dc7f-5332-44a2-bb52-28901b78a7e3/cd40e0a1-5e03-48e1-9b54-a7b8526d72ef"
-					(reference "D8")
-					(unit 1)
-				)
-				(path "/9942a424-e19d-4ffb-8473-f960b5c811cf/db59dc7f-5332-44a2-bb52-28901b78a7e3/f4a90ec5-c194-4316-a05a-ec25706dc995"
-					(reference "D10")
+				(path "/9942a424-e19d-4ffb-8473-f960b5c811cf/db59dc7f-5332-44a2-bb52-28901b78a7e3/f4a90ec5-c194-4316-a05a-ec25706dc995"
+					(reference "D7")
 					(unit 1)
 				)
@@
 		(dnp no)
 		(fields_autoplaced yes)
-		(property "Reference" "Q10"
+		(property "Reference" "Q2"
 			(at 152.4 80.0099 0)
 			(effects
@@
 			(project ""
 				(path "/9942a424-e19d-4ffb-8473-f960b5c811cf/db59dc7f-5332-44a2-bb52-28901b78a7e3/57d5af05-edab-40f7-aafe-6a2e0130ba84"
-					(reference "Q10")
-					(unit 1)
-				)
-				(path "/9942a424-e19d-4ffb-8473-f960b5c811cf/db59dc7f-5332-44a2-bb52-28901b78a7e3/b88b6ec3-afc4-43aa-baa2-21af531f917d"
-					(reference "Q11")
-					(unit 1)
-				)
-				(path "/9942a424-e19d-4ffb-8473-f960b5c811cf/db59dc7f-5332-44a2-bb52-28901b78a7e3/cd40e0a1-5e03-48e1-9b54-a7b8526d72ef"
-					(reference "Q12")
-					(unit 1)
-				)
-				(path "/9942a424-e19d-4ffb-8473-f960b5c811cf/db59dc7f-5332-44a2-bb52-28901b78a7e3/f4a90ec5-c194-4316-a05a-ec25706dc995"
-					(reference "Q13")
-					(unit 1)
-				)
+					(reference "Q2")
+					(unit 1)
+				)
+				(path "/9942a424-e19d-4ffb-8473-f960b5c811cf/db59dc7f-5332-44a2-bb52-28901b78a7e3/b88b6ec3-afc4-43aa-baa2-21af531f917d"
+					(reference "Q4")
+					(unit 1)
+				)
+				(path "/9942a424-e19d-4ffb-8473-f960b5c811cf/db59dc7f-5332-44a2-bb52-28901b78a7e3/cd40e0a1-5e03-48e1-9b54-a7b8526d72ef"
+					(reference "Q6")
+					(unit 1)
+				)
+				(path "/9942a424-e19d-4ffb-8473-f960b5c811cf/db59dc7f-5332-44a2-bb52-28901b78a7e3/f4a90ec5-c194-4316-a05a-ec25706dc995"
+					(reference "Q8")
+					(unit 1)
+				)
