File: BDUCU/voltage regulator.kicad_sch (KiCad schematic)
At the start: 13 parts, among them U17 TPS54302

Commit message: bomupdates
Parts:
- C39: Price (none) -> 0.375
- L1: Price (none) -> .35
- U17: Price (none) -> .93
Changed lines of the file:
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@@
+			"AAAAAAAAAAAAAAAAAAAAAAAAAAAAAAAAAAAAAAAAAAAAAAAAAAAAAAAAAAAAAAAAAAAAAAAAAAAA"
+			"AAAAAAAAAAAAAAAAAAAAAAAAAAAAAAAAAAAAAAAAAAAAAAAAAAAAAAAAAAAAAAAAAAAAAAAAAAAA"
+			"AAAAAAAAAAAAAAAAAAAAAAAAAAAAAAAAAAAAAAAAAAAAAAAAAAAAAAAAAAAAAAAAAAAAAAAAAAAA"
+			"AAAAAAAAAAAAAAAAAAAAAAAAAAAAAAAAAAAAAAAAAAAAAAAAAAAAAAAAAAAAAAAAAAAAAAAAAAAA"
+			"AAAAAAAAAAAAAAAAAAAAAAAAAAAAAAAAAAAAAAAAAAAAAAAAAAAAAAAAAAAAAAAAAAAAAAAAAAAA"
+			"AAAAAAAAAAAAAAAAAAAAAAAAAAAAAAAAAAAAAAAAAAAAAAAAAAAAAAAAAAAAAAAAAAAAAAAAAAAA"
+			"AAAAAAAAAAAAAAAAAAAAAAAAAAAAAAAAAAAAAAAAAAAAAAAAAAAAAAAAAAAAAAAAAAAAAAAAAAAA"
+			"AAAAAAAAAAAAAAAAAAAAAAAAAAAAAAAAAAAAAAAAAAAAAAAAAAAAAAAAAAAAAAAAAAAAAAAAAAAA"
+			"AAAAAAAAAAAAAAAAAAAAAAAAAAAAAAAAAAAAAAAAAAAAAAAAAAAAAAAAAAAAAAAAAAAAAAAAAAAA"
+			"AAAAAAAAAAAAAAAAAAAAAAAAAAAAAAAAAAAAAAAAAAAAAAAAAAAAAAAAAAAAAAAAAAAAAAAAAAAA"
+			"AAAAAAAAAAAAAAAAAAAAAAAAAAAAAAAAAAAAAAAAAAAAAAAAAAAAAAAAAAAAAAAAAAAAAAAAAAAA"
+			"AAAAAAAAAAAAAAAAAAAAAAAAAAAAAAAAAAAAAAAAAAAAAAAAAAAAAAAAAAAAAAAAAAAAAAAAAAAA"
+			"AAAAAAAAAAAAAAAAAAAAAAAAAAAAAAAAAAAAAAAAAAAAAAAAAAAAAAAAAAAAAAAAAAAAAAAAAAAA"
+			"AAAAAAAAAAAAAAAAAAAAAAAAAAAAAAAAAAAAAAAAAAAAAAAAAAAAAAAAAAAAAAAAAAAAAAAAAAAA"
+			"AAAAAAAAAAAAAAAAAAAAAAAAAAAAAAAAAAAAAAAAAAAAAAAAAAAAAAAAAAAAAAAAAAAAAAAAAAAA"
+			"AAAAAAAAAAAAAAAAAAAAAAAAAAAAAAAAAAAAAAAAAAAAAAAAAAAAAAAAAAAAAAAAAAAAAAAAAAAA"
+			"AAAAAAAAAAAAAAAAAAAAAAAAAAAAAAAAAAAAAAAAAAAAAAAAAAAAAAAAAAAAAAAAAAAAAAAAAAAA"
+			"AAAAAAAAAAAAAAAAAAAAAAAAAAAAAAAAAAAAAAAAAAAAAAAAAAAAAAAAAAAAAAAAAAAAAAAAAAAA"
+			"AAAAAAAAAAAAAAAAAAAAAAAAAAAAAAAAAAAAAAAAAAAAAAAAAAAAAAAAAAAAAAAAAAAAAAAAAAAA"
+			"AAAAAAAAAAAAAAAAAAAAAAAAAAAAAAAAAAAAAAAAAAAAAAAAAAAAAAAAAAAAAAAAAAAAAAAAAAAA"
+			"AAAAAAAAAAAAAAAAAAAAAAAAAAAAAAAAAAAAAAAAAAAAAAAAAAAAAAAAAAAAAAAAAAAAAAAAAAAA"
+			"AAAAAAAAAAAAAAAAAAAAAAAAAAAAAAAAAAAAAAAAAAAAAAAAAAAAAAAAAAAAAAAAAAAAAAAAAAAA"
+			"AAAAAAAAAAAAAAAAAAAAAAAAAAAAAAAAAAAAAAAAAAAAAAAAAAAAAAAAAAAAAAAAAAAAAAAAAAAA"
+			"AAAAAAAAAAAAAAAAAAAAAAAAAAAAAAAAAAAAAAAAAAAAAAAAAAAAAAAAAAAAAAAAAAAAAAAAAAAA"
+			"AAAAAAAAAAAAAAAAAAAAAAAAAAAAAAAAAAAAAAAAAAAAAAAAAAAAAAAAAAAAAAAAAAAAAAAAAAAA"
+			"AAAAAAAAAAAAAAAAAAAAAAAAAAAAAAAAAAAAAAAAAAAAAAAAAAAAAAAAAAAAAAAAAAAAAAAAAAAA"
+			"AAAAAAAAAAAAAAAAAAAAAAAAAAAAAAAAAAAAAAAAAAAAAAAAAAAAAAAAAAAAAAAAAAAAAAAAAAAA"
+			"AAAAAAAAAAAAAAAAAAAAAAAAAAAAAAAAAAAAAAAAAAAAAAAAAAAAAAAAAAAAAAAAAAAAAAAAAAAA"
+			"AAAAAAAAAAAAAAAAAAAAAAAAAAAAAAAAAAAAAAAAAAAAAAAAAAAAAAAAAAAAAAAAAAAAAAAAAAAA"
+			"AAAAAAAAAAAAAAAAAAAAAAAAAAAAAAAAAAAAAAAAAAAAAAAAAAAAAAAAAAAAAAAAAAAAAAAAAAAA"
+			"AAAAAAAAAAAAAAAAAAAAAAAAAAAAAAAAAAAAAAAAAAAAAAAAAAAAAAAAAAAAAAAAAAAAAAAAAAAA"
+			"AAAAAAAAAAAAAAAAAAAAAAAAAAAAAAAAAAAAAAAAAAAAAAAAAAAAAAAAAAAAAAAAAAAAAAAAAAAA"
+			"AAAAAAAAAAAAAAAAAAAAAAAAAAAAAAAAAAAAAAAAAAAAAAAAAAAAAAAAAAAAAAAAAAAAAAAAAAAA"
+			"AAAAAAAAAAAAAAAAAAAAAAAAAAAAAAAAAAAAAAAAAAAAAAAAAAAAAAAAAAAAAAAAAAAAAAAAAAAA"
+			"AAAAAAAAAAAAAAAAAAAAAAAAAAAAAAAAAAAAAAAAAAAAAAAAAAAAAAAAAAAAAAAAAAAAAAAAAAAA"
+			"AAAAAAAAAAAAAAAAAAAAAAAAAAAAAAAAAAAAAAAAAAAAAAAAAAAAAAAAAAAAAAAAAAAAAAAAAAAA"
 			"AAAAAAAAAAAAAAAAAAAAAAAAAAAAAAAAAAAAAAAAAAAAAAAAAAAAAAAAAAAAAAAAAAAAAAAAAAAA"
 			"AAAAAAAAAAAAAAAAAAAAAAAAAAAAAAAAAAAAAAAAAAAAAAAAAAAAAAAAAAAAAAAAAAAAAAAAAAAA"
@@
 			"AAAAAAAAAAAAAAAAAAAAAAAAAAAAAAAAAAAAAAAAAAAAAAAAAAAAAAAAAAAAAAAAAAAAAAAAAAAA"
 			"AAAAAAAAAAAAAAAAAAAAAAAAAAAAAAAAAAAAAAAAAAAAAAAAAAAAAAAAAAAAAAAAAAAAAAAAAAAA"
-			"AAAAAAAAAAAAAAAAAAAAAAAAAA=="
+			"AAAAAAAAAAAAAAAAAAAAAAAAAAEBABcGgQEQAQEAGwMBEBABAQAdBQFAEAEBABYFwQAQAQEAAQZA"
+			"ABABAQAbAwEQEAEBABwFATAQAQEAFgWBABABAQAaBgEMEAEBABsDARAQAQEAFAYxABABAQAXBQEB"
+			"EAEBAAMGRAASAQ0AEwERABMBGQAYAQEDGgEBCBkCAQYaAQEIEgMJABoBAQgZAgEGGgEBCBsDARgT"
+			"AREAGAEBAhgCAQMSAw0AGwIBGBoDAQgYAgEDGQMBBBsCARgSBAkAGAIBAxIDDQAbAgEYGgMBCBgC"
+			"AQMZAwEEGwIBGBkEAQYAAAAAAAAAAAAAAAAAAAAAAAAAAAAAAAAAaXThtAEAAAAAAAAAAAAAAAAA"
+			"AAAAAAAPAAAAAAAAAAB0YWxpYwAAAAAAAAAAAAAAAAAAAAAAAA8AAAAAAAAAAGVqYVZ1IFNlcmlm"
+			"AAAAAAAAAAAAAAAADwAAAAAAAAAAAAAAAAAAAAAAAAAAAAAAAAAAAAAAAAAAgHThtAEAAAAAAAAA"
+			"AAAAAAAAAAAAAAAPAAAAAAAAAABvbGQgSXRhbGljAAAAAAAAAAAAAAAAAA8AAAAAAAAAAGVqYVZ1"
+			"IFNlcmlmAAAAAAAAAAAAAAAADwAAAAAAAAAAAAAAAAAAAAAAAAAAAAAAAAAAAAAAAADTAAHSjhOG"
+			"EAB6zOG0AQAAAAAAAAAAAAAAAAAAAAAAAA8AAAAAAAAAAHRhbGljAAAAAAAAAAAAAAAAAAAAAAAA"
+			"DwAAAAAAAAAAZW9yZ2lhAAAAAAAAAAAAAAAAAAAAAAAPAAAAAAAAAAAAAAAAAAAAAAAAAAAAAAAA"
+			"AAAAAAAAAACfzOG0AQAAAAAAAAAAAAAAAAAAAAAAAA8AAAAAAAAAAGVndWxhcgAAAAAAAAAAAAAA"
+			"AAAAAAAADwAAAAAAAAAAZW9yZ2lhAAAAAAAAAAAAAAAAAAAAAAAPAAAAAAAAAAAAAAAAAAAAAAAA"
+			"AAAAAAAAAAAAAAAAAACbzOG0AQAAAAAAAAAAAAAAAAAAAAAAAA8AAAAAAAAAAG9sZCBJdGFsaWMA"
+			"AAAAAAAAAAAAAAAADwAAAAAAAAAAZW9yZ2lhAAAAAAAAAAAAAAAAAAAAAAAPAAAAAAAAAAAAAAAA"
+			"AAAAAAAAAAAAAAAAAAAAAAAAAADK5fa0AQAAAAAAAAAAAAAAAAAAAAAAAA8AAAAAAAAAAG9sZAAA"
+			"AAAAAAAAAAAAAAAAAAAAAAAADwAAAAAAAAAAZW9yZ2lhAAAAAAAAAAAAAAAAAAAAAAAPAAAAAAAA"
+			"AAAAAAAAAAAAAAAAAAAAAAAAAAAAAAAAAADU5fa0AQAAAAAAAAAAAAAAAAAAAAAAAA8AAAAAAAAA"
+			"AHRhbGljAAAAAAAAAAAAAAAAAAAAAAAAnayMpwAWAYAAYHjzigEAAJysjacAFwGAAAAAAAAAAACf"
+			"rLKnABgBgABlbWlMaWdonqyzpwAZAYAAAAAAAAAAAJGssKcAGgGAAG90byBTYW6QrLGnABsBgAAA"
+			"AAAAAAAAk6y2pwAcAYAAAAAAAAAAAJKst6cAHQGAAAAAAAAAAACVrLSnih4BgAAAAAAAAAAAlKy1"
+			"pwAfAYAPAAAAAAAAAJesuqcAIAGAAAAAAAAAAACWrLunACEBgA8AAAAAAAAAiay4pyAiAYBzIEhL"
+			"AAAAAIisuacAIwGADwAAAAAAAACLrL6nACQBgAAAAAAAAAAAiqy/pwAlAYAAX3jzigEAAI2svKcA"
+			"JgGAAAAAAAAAAACMrL2nACcBgABpZ2h0AAAAj6yipwAoAYAAAAAAAAAAAI6so6cAKQGAAG90byBT"
+			"YW6BrKCnACoBgAAAAAAAAAAAgKyhpwArAYAAAAAAAAAAAIOspqcALAGAAAAAAAAAAACCrKenii0B"
+			"gAAAAAAAAAAAhaykpwAuAYAPAAAAAAAAAISspacALwGAAAAAAAAAAACHrKqnADABgA8AAAAAAAAA"
+			"hqyrpyAxAYBzIEhLAAAAAPmsqKcAMgGADwAAAAAAAAD4rKmnADMBgAAAAAAAAAAA+6yupwA0AYAA"
+			"AAAAAAAAAPqsr6c0NQGAUAFk1YoBAAD9rKynijYBgAAAAAAAAAAA/Kytp4o3AYAAJk3cigEAAP+s"
+			"0qcAOAGAAAAAAAAAAAD+rNOnADkBgABvbGQgQ29u8azQp2U6AYAAAAAAAAAAAPCs0acAOwGAAGFo"
+			"bnNjaHLzrNanADwBgAAAAAAAAAAA8qzXpwA9AYAAAAAAAAAAAPWs1KcAPgGAAAAAAAAAAAD0rNWn"
+			"ij8BgAAAAAAAAAAA96zapwBAAYAPAAAAAAAAAPas26eKQQGAAAAAAAAAAADprNinAEIBgA8AAAAA"
+			"AAAA6KzZp3NDAYBpZnQAAAAAAOus3qcARAGADwAAAAAAAADqrN+nAEUBgAAAAAAAAAAA7azcpwBG"
+			"AYAAQE3cigEAAOys3acARwGAAAAAAAAAAADvrMKnAEgBgABlZ3VsYXIA7qzDpwBJAYAAAAAAAAAA"
+			"AOGswKcASgGAAGFobnNjaHLgrMGnAEsBgAAAAAAAAAAA46zGpwBMAYAAAAAAAAAAAOKsx6cATQGA"
+			"AAAAAAAAAADlrMSnik4BgAAAAAAAAAAA5KzFpwBPAYAPAAAAAAAAAOesyqeKUAGAAAAAAAAAAADm"
+			"rMunAFEBgA8AAAAAAAAA2azIp3NSAYBpZnQAAAAAANisyacAUwGADwAAAAAAAADbrM6nAFQBgAAA"
+			"AAAAAAAA2qzPpwBVAYAANE3cig=="
 		)
 	)
@@
 		(on_board yes)
 		(dnp no)
-		(property "Reference" "#PWR?"
+		(property "Reference" "#PWR0106"
 			(at 190.5 104.14 0)
 			(effects
@@
 		(on_board yes)
 		(dnp no)
-		(property "Reference" "#PWR?"
+		(property "Reference" "#PWR0109"
 			(at 201.93 88.9 0)
 			(effects
@@
 		(dnp no)
 		(fields_autoplaced yes)
-		(property "Reference" "C?"
+		(property "Reference" "C35"
 			(at 171.45 76.5809 0)
 			(effects
@@
 		(dnp no)
 		(fields_autoplaced yes)
-		(property "Reference" "#PWR?"
+		(property "Reference" "#PWR0104"
 			(at 212.09 78.74 0)
 			(effects
@@
 		(on_board yes)
 		(dnp no)
-		(property "Reference" "C?"
+		(property "Reference" "C36"
 			(at 104.14 74.0409 0)
 			(effects
@@
 		(dnp no)
 		(fields_autoplaced yes)
-		(property "Reference" "#PWR?"
+		(property "Reference" "#PWR0108"
 			(at 173.99 88.9 0)
 			(effects
@@
 		(dnp no)
 		(fields_autoplaced yes)
-		(property "Reference" "U?"
+		(property "Reference" "U17"
 			(at 137.16 64.77 0)
 			(effects
@@
 			)
 		)
+		(property "Price" ".93"
+			(at 137.16 74.93 0)
+			(effects
+				(font
+					(size 1.27 1.27)
+				)
+			)
+		)
 		(pin "5"
 		)
@@
 		(dnp no)
 		(fields_autoplaced yes)
-		(property "Reference" "R?"
+		(property "Reference" "R74"
 			(at 193.04 85.0899 0)
 			(effects
@@
 		(dnp no)
 		(fields_autoplaced yes)
-		(property "Reference" "L?"
+		(property "Reference" "L1"
 			(at 160.02 69.85 90)
 			(effects
@@
 			)
 		)
+		(property "Price" ".35"
+			(at 160.02 74.93 0)
+			(effects
+				(font
+					(size 1.27 1.27)
+				)
+			)
+		)
 		(pin "1"
 		)
@@
 		(dnp no)
 		(fields_autoplaced yes)
-		(property "Reference" "#PWR?"
+		(property "Reference" "#PWR0102"
 			(at 93.98 76.2 0)
 			(effects
@@
 		(dnp no)
 		(fields_autoplaced yes)
-		(property "Reference" "#PWR?"
+		(property "Reference" "#PWR0103"
 			(at 137.16 91.44 0)
 			(effects
@@
 		(dnp no)
 		(fields_autoplaced yes)
-		(property "Reference" "C?"
+		(property "Reference" "C38"
 			(at 205.74 77.4699 0)
 			(effects
@@
 		(dnp no)
 		(fields_autoplaced yes)
-		(property "Reference" "C?"
+		(property "Reference" "C37"
 			(at 118.11 74.9299 0)
 			(effects
@@
 		(dnp no)
 		(fields_autoplaced yes)
-		(property "Reference" "F?"
+		(property "Reference" "F7"
 			(at 205.74 68.58 90)
 			(effects
@@
 		(dnp no)
 		(fields_autoplaced yes)
-		(property "Reference" "C?"
+		(property "Reference" "C34"
 			(at 151.13 64.77 90)
 			(effects
@@
 		(dnp no)
 		(fields_autoplaced yes)
-		(property "Reference" "R?"
+		(property "Reference" "R73"
 			(at 193.04 77.4699 0)
 			(effects
@@
 		(dnp no)
 		(fields_autoplaced yes)
-		(property "Reference" "C?"
+		(property "Reference" "C40"
 			(at 182.88 76.5809 0)
 			(effects
@@
 		(on_board yes)
 		(dnp no)
-		(property "Reference" "C?"
+		(property "Reference" "C39"
 			(at 90.17 74.0409 0)
 			(effects
@@
 			)
 		)
+		(property "Price" "0.375"
+			(at 93.98 76.2 0)
+			(effects
+				(font
+					(size 1.27 1.27)
+				)
+			)
+		)
 		(pin "1"
 		)
@@
 		(dnp no)
 		(fields_autoplaced yes)
-		(property "Reference" "R?"
+		(property "Reference" "R75"
 			(at 193.04 92.7099 0)
 			(effects

Commit message: I am Nicholas Chan (lesbian version)
Parts:
- renumbered C39 to C36, C36 to C37, C37 to C38, C34 to C39, C35 to C40, C40 to C41, C38 to C42, F7 to F3, U17 to U18
Changed lines of the file:
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@@
 		(on_board yes)
 		(dnp no)
-		(property "Reference" "#PWR0106"
+		(property "Reference" "#PWR0127"
 			(at 190.5 104.14 0)
 			(effects
@@
 			(project "BDUCU"
 				(path "/9942a424-e19d-4ffb-8473-f960b5c811cf/d4ffcd89-988d-4b7a-a40c-cc22466602f9"
-					(reference "#PWR0106")
+					(reference "#PWR0127")
 					(unit 1)
 				)
@@
 		(on_board yes)
 		(dnp no)
-		(property "Reference" "#PWR0109"
+		(property "Reference" "#PWR0128"
 			(at 201.93 88.9 0)
 			(effects
@@
 			(project "BDUCU"
 				(path "/9942a424-e19d-4ffb-8473-f960b5c811cf/d4ffcd89-988d-4b7a-a40c-cc22466602f9"
-					(reference "#PWR0109")
+					(reference "#PWR0128")
 					(unit 1)
 				)
@@
 		(dnp no)
 		(fields_autoplaced yes)
-		(property "Reference" "C35"
+		(property "Reference" "C40"
 			(at 171.45 76.5809 0)
 			(effects
@@
 			(project ""
 				(path "/9942a424-e19d-4ffb-8473-f960b5c811cf/d4ffcd89-988d-4b7a-a40c-cc22466602f9"
-					(reference "C35")
+					(reference "C40")
 					(unit 1)
 				)
@@
 		(dnp no)
 		(fields_autoplaced yes)
-		(property "Reference" "#PWR0104"
+		(property "Reference" "#PWR0129"
 			(at 212.09 78.74 0)
 			(effects
@@
 			(project ""
 				(path "/9942a424-e19d-4ffb-8473-f960b5c811cf/d4ffcd89-988d-4b7a-a40c-cc22466602f9"
-					(reference "#PWR0104")
+					(reference "#PWR0129")
 					(unit 1)
 				)
@@
 		(on_board yes)
 		(dnp no)
-		(property "Reference" "C36"
+		(property "Reference" "C37"
 			(at 104.14 74.0409 0)
 			(effects
@@
 			(project "BDUCU"
 				(path "/9942a424-e19d-4ffb-8473-f960b5c811cf/d4ffcd89-988d-4b7a-a40c-cc22466602f9"
-					(reference "C36")
+					(reference "C37")
 					(unit 1)
 				)
@@
 		(dnp no)
 		(fields_autoplaced yes)
-		(property "Reference" "#PWR0108"
+		(property "Reference" "#PWR0126"
 			(at 173.99 88.9 0)
 			(effects
@@
 			(project "BDUCU"
 				(path "/9942a424-e19d-4ffb-8473-f960b5c811cf/d4ffcd89-988d-4b7a-a40c-cc22466602f9"
-					(reference "#PWR0108")
+					(reference "#PWR0126")
 					(unit 1)
 				)
@@
 		(dnp no)
 		(fields_autoplaced yes)
-		(property "Reference" "U17"
+		(property "Reference" "U18"
 			(at 137.16 64.77 0)
 			(effects
@@
 			(project ""
 				(path "/9942a424-e19d-4ffb-8473-f960b5c811cf/d4ffcd89-988d-4b7a-a40c-cc22466602f9"
-					(reference "U17")
+					(reference "U18")
 					(unit 1)
 				)
@@
 		(dnp no)
 		(fields_autoplaced yes)
-		(property "Reference" "#PWR0102"
+		(property "Reference" "#PWR0124"
 			(at 93.98 76.2 0)
 			(effects
@@
 			(project ""
 				(path "/9942a424-e19d-4ffb-8473-f960b5c811cf/d4ffcd89-988d-4b7a-a40c-cc22466602f9"
-					(reference "#PWR0102")
+					(reference "#PWR0124")
 					(unit 1)
 				)
@@
 		(dnp no)
 		(fields_autoplaced yes)
-		(property "Reference" "#PWR0103"
+		(property "Reference" "#PWR0125"
 			(at 137.16 91.44 0)
 			(effects
@@
 			(project ""
 				(path "/9942a424-e19d-4ffb-8473-f960b5c811cf/d4ffcd89-988d-4b7a-a40c-cc22466602f9"
-					(reference "#PWR0103")
+					(reference "#PWR0125")
 					(unit 1)
 				)
@@
 		(dnp no)
 		(fields_autoplaced yes)
-		(property "Reference" "C38"
+		(property "Reference" "C42"
 			(at 205.74 77.4699 0)
 			(effects
@@
 			(project "BDUCU"
 				(path "/9942a424-e19d-4ffb-8473-f960b5c811cf/d4ffcd89-988d-4b7a-a40c-cc22466602f9"
-					(reference "C38")
+					(reference "C42")
 					(unit 1)
 				)
@@
 		(dnp no)
 		(fields_autoplaced yes)
-		(property "Reference" "C37"
+		(property "Reference" "C38"
 			(at 118.11 74.9299 0)
 			(effects
@@
 			(project "BDUCU"
 				(path "/9942a424-e19d-4ffb-8473-f960b5c811cf/d4ffcd89-988d-4b7a-a40c-cc22466602f9"
-					(reference "C37")
+					(reference "C38")
 					(unit 1)
 				)
@@
 		(dnp no)
 		(fields_autoplaced yes)
-		(property "Reference" "F7"
+		(property "Reference" "F3"
 			(at 205.74 68.58 90)
 			(effects
@@
 			(project ""
 				(path "/9942a424-e19d-4ffb-8473-f960b5c811cf/d4ffcd89-988d-4b7a-a40c-cc22466602f9"
-					(reference "F7")
+					(reference "F3")
 					(unit 1)
 				)
@@
 		(dnp no)
 		(fields_autoplaced yes)
-		(property "Reference" "C34"
+		(property "Reference" "C39"
 			(at 151.13 64.77 90)
 			(effects
@@
 			(project ""
 				(path "/9942a424-e19d-4ffb-8473-f960b5c811cf/d4ffcd89-988d-4b7a-a40c-cc22466602f9"
-					(reference "C34")
+					(reference "C39")
 					(unit 1)
 				)
@@
 		(dnp no)
 		(fields_autoplaced yes)
-		(property "Reference" "C40"
+		(property "Reference" "C41"
 			(at 182.88 76.5809 0)
 			(effects
@@
 			(project "BDUCU"
 				(path "/9942a424-e19d-4ffb-8473-f960b5c811cf/d4ffcd89-988d-4b7a-a40c-cc22466602f9"
-					(reference "C40")
+					(reference "C41")
 					(unit 1)
 				)
@@
 		(on_board yes)
 		(dnp no)
-		(property "Reference" "C39"
+		(property "Reference" "C36"
 			(at 90.17 74.0409 0)
 			(effects
@@
 			(project "BDUCU"
 				(path "/9942a424-e19d-4ffb-8473-f960b5c811cf/d4ffcd89-988d-4b7a-a40c-cc22466602f9"
-					(reference "C39")
-					(unit 1)
-				)
+					(reference "C36")
+					(unit 1)
+				)
