File: BDUCU/voltage regulator.kicad_sch (KiCad schematic)
At the start: 13 parts, among them U18 TPS54302

Commit message: microsoft ppBDUCU update and changes because nicholas draw wrong stuffs
Parts:
- renumbered C36 to C33, C37 to C34, C38 to C35, C39 to C36, C40 to C37, C41 to C38, C42 to C39, R73 to R68, R74 to R69, R75 to R70, U18 to U17
Changed lines of the file:
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@@
 		(in_pos_files yes)
 		(dnp no)
-		(property "Reference" "#PWR0127"
+		(property "Reference" "#PWR0120"
 			(at 190.5 104.14 0)
 			(hide yes)
@@
 			(project "BDUCU"
 				(path "/9942a424-e19d-4ffb-8473-f960b5c811cf/d4ffcd89-988d-4b7a-a40c-cc22466602f9"
-					(reference "#PWR0127")
+					(reference "#PWR0120")
 					(unit 1)
 				)
@@
 		(in_pos_files yes)
 		(dnp no)
-		(property "Reference" "#PWR0128"
+		(property "Reference" "#PWR0121"
 			(at 201.93 88.9 0)
 			(hide yes)
@@
 			(project "BDUCU"
 				(path "/9942a424-e19d-4ffb-8473-f960b5c811cf/d4ffcd89-988d-4b7a-a40c-cc22466602f9"
-					(reference "#PWR0128")
+					(reference "#PWR0121")
 					(unit 1)
 				)
@@
 		(dnp no)
 		(fields_autoplaced yes)
-		(property "Reference" "C40"
+		(property "Reference" "C37"
 			(at 171.45 76.5809 0)
 			(show_name no)
@@
 			(project "BDUCU"
 				(path "/9942a424-e19d-4ffb-8473-f960b5c811cf/d4ffcd89-988d-4b7a-a40c-cc22466602f9"
-					(reference "C40")
+					(reference "C37")
 					(unit 1)
 				)
@@
 		(dnp no)
 		(fields_autoplaced yes)
-		(property "Reference" "#PWR0129"
+		(property "Reference" "#PWR0122"
 			(at 212.09 78.74 0)
 			(hide yes)
@@
 			(project "BDUCU"
 				(path "/9942a424-e19d-4ffb-8473-f960b5c811cf/d4ffcd89-988d-4b7a-a40c-cc22466602f9"
-					(reference "#PWR0129")
+					(reference "#PWR0122")
 					(unit 1)
 				)
@@
 		(in_pos_files yes)
 		(dnp no)
-		(property "Reference" "C37"
+		(property "Reference" "C34"
 			(at 104.14 74.0409 0)
 			(show_name no)
@@
 			(project "BDUCU"
 				(path "/9942a424-e19d-4ffb-8473-f960b5c811cf/d4ffcd89-988d-4b7a-a40c-cc22466602f9"
-					(reference "C37")
+					(reference "C34")
 					(unit 1)
 				)
@@
 		(dnp no)
 		(fields_autoplaced yes)
-		(property "Reference" "#PWR0126"
+		(property "Reference" "#PWR0119"
 			(at 173.99 88.9 0)
 			(hide yes)
@@
 			(project "BDUCU"
 				(path "/9942a424-e19d-4ffb-8473-f960b5c811cf/d4ffcd89-988d-4b7a-a40c-cc22466602f9"
-					(reference "#PWR0126")
+					(reference "#PWR0119")
 					(unit 1)
 				)
@@
 		(dnp no)
 		(fields_autoplaced yes)
-		(property "Reference" "U18"
+		(property "Reference" "U17"
 			(at 137.16 64.77 0)
 			(show_name no)
@@
 			(project "BDUCU"
 				(path "/9942a424-e19d-4ffb-8473-f960b5c811cf/d4ffcd89-988d-4b7a-a40c-cc22466602f9"
-					(reference "U18")
+					(reference "U17")
 					(unit 1)
 				)
@@
 		(dnp no)
 		(fields_autoplaced yes)
-		(property "Reference" "R74"
+		(property "Reference" "R69"
 			(at 193.04 85.0899 0)
 			(show_name no)
@@
 			(project "BDUCU"
 				(path "/9942a424-e19d-4ffb-8473-f960b5c811cf/d4ffcd89-988d-4b7a-a40c-cc22466602f9"
-					(reference "R74")
+					(reference "R69")
 					(unit 1)
 				)
@@
 		(dnp no)
 		(fields_autoplaced yes)
-		(property "Reference" "#PWR0124"
+		(property "Reference" "#PWR0117"
 			(at 93.98 76.2 0)
 			(hide yes)
@@
 			(project "BDUCU"
 				(path "/9942a424-e19d-4ffb-8473-f960b5c811cf/d4ffcd89-988d-4b7a-a40c-cc22466602f9"
-					(reference "#PWR0124")
+					(reference "#PWR0117")
 					(unit 1)
 				)
@@
 		(dnp no)
 		(fields_autoplaced yes)
-		(property "Reference" "#PWR0125"
+		(property "Reference" "#PWR0118"
 			(at 137.16 91.44 0)
 			(hide yes)
@@
 			(project "BDUCU"
 				(path "/9942a424-e19d-4ffb-8473-f960b5c811cf/d4ffcd89-988d-4b7a-a40c-cc22466602f9"
-					(reference "#PWR0125")
+					(reference "#PWR0118")
 					(unit 1)
 				)
@@
 		(dnp no)
 		(fields_autoplaced yes)
-		(property "Reference" "C42"
+		(property "Reference" "C39"
 			(at 205.74 77.4699 0)
 			(show_name no)
@@
 			(project "BDUCU"
 				(path "/9942a424-e19d-4ffb-8473-f960b5c811cf/d4ffcd89-988d-4b7a-a40c-cc22466602f9"
-					(reference "C42")
+					(reference "C39")
 					(unit 1)
 				)
@@
 		(dnp no)
 		(fields_autoplaced yes)
-		(property "Reference" "C38"
+		(property "Reference" "C35"
 			(at 118.11 74.9299 0)
 			(show_name no)
@@
 			(project "BDUCU"
 				(path "/9942a424-e19d-4ffb-8473-f960b5c811cf/d4ffcd89-988d-4b7a-a40c-cc22466602f9"
-					(reference "C38")
+					(reference "C35")
 					(unit 1)
 				)
@@
 		(dnp no)
 		(fields_autoplaced yes)
-		(property "Reference" "C39"
+		(property "Reference" "C36"
 			(at 151.13 64.77 90)
 			(show_name no)
@@
 			(project "BDUCU"
 				(path "/9942a424-e19d-4ffb-8473-f960b5c811cf/d4ffcd89-988d-4b7a-a40c-cc22466602f9"
-					(reference "C39")
+					(reference "C36")
 					(unit 1)
 				)
@@
 		(dnp no)
 		(fields_autoplaced yes)
-		(property "Reference" "R73"
+		(property "Reference" "R68"
 			(at 193.04 77.4699 0)
 			(show_name no)
@@
 			(project "BDUCU"
 				(path "/9942a424-e19d-4ffb-8473-f960b5c811cf/d4ffcd89-988d-4b7a-a40c-cc22466602f9"
-					(reference "R73")
+					(reference "R68")
 					(unit 1)
 				)
@@
 		(dnp no)
 		(fields_autoplaced yes)
-		(property "Reference" "C41"
+		(property "Reference" "C38"
 			(at 182.88 76.5809 0)
 			(show_name no)
@@
 			(project "BDUCU"
 				(path "/9942a424-e19d-4ffb-8473-f960b5c811cf/d4ffcd89-988d-4b7a-a40c-cc22466602f9"
-					(reference "C41")
+					(reference "C38")
 					(unit 1)
 				)
@@
 		(in_pos_files yes)
 		(dnp no)
-		(property "Reference" "C36"
+		(property "Reference" "C33"
 			(at 90.17 74.0409 0)
 			(show_name no)
@@
 			(project "BDUCU"
 				(path "/9942a424-e19d-4ffb-8473-f960b5c811cf/d4ffcd89-988d-4b7a-a40c-cc22466602f9"
-					(reference "C36")
+					(reference "C33")
 					(unit 1)
 				)
@@
 		(dnp no)
 		(fields_autoplaced yes)
-		(property "Reference" "R75"
+		(property "Reference" "R70"
 			(at 193.04 92.7099 0)
 			(show_name no)
@@
 			(project "BDUCU"
 				(path "/9942a424-e19d-4ffb-8473-f960b5c811cf/d4ffcd89-988d-4b7a-a40c-cc22466602f9"
-					(reference "R75")
-					(unit 1)
-				)
+					(reference "R70")
+					(unit 1)
+				)
