File: BDUCU/hall_isense.kicad_sch (KiCad schematic)
At the start: 6 parts, among them U8 LM358, U9 LM358

Commit message: microsoft ppBDUCU update and changes because nicholas draw wrong stuffs
Connections:
- net PRE_R_T: now also U9.6 (-), U9.7; no longer U9.1, U9.2 (-)
- net PRE_R_T_input: now also U9.5 (+); no longer U9.3 (+)
- net TS-_T: now also U9.1, U9.2 (-); no longer U9.6 (-), U9.7
- net TS-_T_input: now also U9.3 (+); no longer U9.5 (+)
Changed lines of the file:
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@@
 		(dnp no)
 		(fields_autoplaced yes)
-		(property "Reference" "#PWR031"
+		(property "Reference" "#PWR030"
 			(at 149.86 59.69 0)
 			(hide yes)
@@
 			(project "BDUCU"
 				(path "/9942a424-e19d-4ffb-8473-f960b5c811cf/6945656a-1a27-4b96-8a88-6a11e7484dc7"
-					(reference "#PWR031")
+					(reference "#PWR030")
 					(unit 1)
 				)
@@
 		(lib_id "Amplifier_Operational:LM358")
 		(at 175.26 100.33 0)
-		(unit 1)
+		(unit 2)
 		(body_style 1)
 		(exclude_from_sim no)
@@
 				(path "/9942a424-e19d-4ffb-8473-f960b5c811cf/6945656a-1a27-4b96-8a88-6a11e7484dc7"
 					(reference "U9")
-					(unit 1)
+					(unit 2)
 				)
 			)
@@
 		(lib_id "Amplifier_Operational:LM358")
 		(at 175.26 120.65 0)
-		(unit 2)
+		(unit 1)
 		(body_style 1)
 		(exclude_from_sim no)
@@
 				(path "/9942a424-e19d-4ffb-8473-f960b5c811cf/6945656a-1a27-4b96-8a88-6a11e7484dc7"
 					(reference "U9")
-					(unit 2)
+					(unit 1)
 				)
 			)
@@
 		(dnp no)
 		(fields_autoplaced yes)
-		(property "Reference" "#PWR032"
+		(property "Reference" "#PWR031"
 			(at 157.48 111.76 0)
 			(hide yes)
@@
 			(project "BDUCU"
 				(path "/9942a424-e19d-4ffb-8473-f960b5c811cf/6945656a-1a27-4b96-8a88-6a11e7484dc7"
-					(reference "#PWR032")
+					(reference "#PWR031")
 					(unit 1)
 				)
@@
 		(dnp no)
 		(fields_autoplaced yes)
-		(property "Reference" "#PWR033"
+		(property "Reference" "#PWR032"
 			(at 157.48 132.08 0)
 			(hide yes)
@@
 			(project "BDUCU"
 				(path "/9942a424-e19d-4ffb-8473-f960b5c811cf/6945656a-1a27-4b96-8a88-6a11e7484dc7"
-					(reference "#PWR033")
+					(reference "#PWR032")
 					(unit 1)
 				)
@@
 		(dnp no)
 		(fields_autoplaced yes)
-		(property "Reference" "#PWR030"
+		(property "Reference" "#PWR029"
 			(at 149.86 41.91 0)
 			(hide yes)
@@
 			(project "BDUCU"
 				(path "/9942a424-e19d-4ffb-8473-f960b5c811cf/6945656a-1a27-4b96-8a88-6a11e7484dc7"
-					(reference "#PWR030")
+					(reference "#PWR029")
 					(unit 1)
 				)
@@
 		(dnp no)
 		(fields_autoplaced yes)
-		(property "Reference" "#PWR035"
+		(property "Reference" "#PWR034"
 			(at 208.915 90.17 0)
 			(hide yes)
@@
 			(project "BDUCU"
 				(path "/9942a424-e19d-4ffb-8473-f960b5c811cf/6945656a-1a27-4b96-8a88-6a11e7484dc7"
-					(reference "#PWR035")
+					(reference "#PWR034")
 					(unit 1)
 				)
@@
 		(dnp no)
 		(fields_autoplaced yes)
-		(property "Reference" "#PWR034"
+		(property "Reference" "#PWR033"
 			(at 208.915 72.39 0)
 			(hide yes)
@@
 			(project "BDUCU"
 				(path "/9942a424-e19d-4ffb-8473-f960b5c811cf/6945656a-1a27-4b96-8a88-6a11e7484dc7"
-					(reference "#PWR034")
+					(reference "#PWR033")
 					(unit 1)
 				)
