File: BDUCU/BDUCU.kicad_pcb (KiCad board)
At the start: 2 copper layers, 140 x 60 mm, 176 parts, among them J1 Conn_01x02_Pin, J10 Conn_02x04_Top_Bottom, J11 Conn_02x02_Top_Bottom, J2 Conn_01x02_Pin, J3 Conn_01x02_Pin, J4 Conn_01x02_Pin, J5 Conn_02x04_Top_Bottom, J6 AIR, J7 Conn_01x02, J9 Conn_02x02_Top_Bottom, Q1 MMBT3906, Q2 AO3400A, Q3 MMBT3906, Q4 AO3400A, Q5 MMBT3906, Q6 AO3400A, Q7 MMBT3906, Q8 AO3400A, SW1 SW_Push, U1 SGM722, U10 MCP2515-xST, U11 TJA1050T_CM_118, U12 ATmega328-A, U13 MCP2515-xST, U14 TJA1050T_CM_118, U15 40106, U16 LTV-847S, U17 TPS54302, U2 SGM722, U7 LM358, U8 LM358, U9 LM358, Y1 20MHz, Y2 16MHz, Y3 20MHz

Commit message: hi
Parts:
- removed J5: Conn_02x04_Top_Bottom, Connector_Molex:Molex_Micro-Fit_3.0_43045-0800_2x04_P3.00mm_Horizontal
- removed J9: Conn_02x02_Top_Bottom, Connector_Molex:Molex_Micro-Fit_3.0_43045-0400_2x02_P3.00mm_Horizontal
- added J12: Conn_02x02_Top_Bottom, Connector_Molex:Molex_Micro-Fit_3.0_43045-0400_2x02_P3.00mm_Horizontal, F.Cu at (146.3, 50.0)
- added J13: Conn_02x02_Top_Bottom, Connector_Molex:Molex_Micro-Fit_3.0_43045-0400_2x02_P3.00mm_Horizontal, F.Cu at (162.5, 50.0)
- C20, CA2, CA3, CA4, CA5, D10, D11, D5, D7, Q3, Q4, Q7, Q8, R35, R36, R37, R38, R43, R44, R45, R46, R52, R53, R54, U15, U16: moved to F.Cu
- C21, CA1, D4, D6, D8, D9, Q1, Q2, Q5, Q6, R24, R31, R32, R33, R34, R39, R40, R41, R42, R48, R50, R55, R56, R57, R58, R59, R60, R61, R62, R63, R64, R65, R66, R67: moved to B.Cu
- moved CA1 73.3 mm to (210.2, 70.2)
- moved R62 69.2 mm to (208.2, 70.2)
- moved D10 69.2 mm to (208.2, 59.1), turned to 180 degrees
- moved CA2 68.7 mm to (207.9, 63.3), turned to 180 degrees
- moved R53 68.7 mm to (207.9, 61.2), turned to 180 degrees
- moved R56 68.7 mm to (207.9, 63.3), turned to 0 degrees
- moved R63 65.2 mm to (206.2, 70.2)
- moved U15 64.2 mm to (205.7, 69.2)
- moved R60 61.2 mm to (204.2, 70.2)
- moved D11 59.8 mm to (203.4, 59.1), turned to 180 degrees
- moved CA5 59.4 mm to (203.2, 63.3), turned to 180 degrees
- moved R58 59.4 mm to (203.2, 63.3), turned to 0 degrees
- moved R54 59.3 mm to (203.2, 61.2), turned to 180 degrees
- moved R61 57.3 mm to (202.2, 70.2)
- moved D9 50.9 mm to (199.0, 59.1), turned to 180 degrees
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Connections:
- J10 pad 1: CAN0_H -> SDC_IN
- J10 pad 2: CAN0_L -> GND
- J10 pad 3: GND -> ~{TS_ACT}
- J10 pad 4: SDC_IN -> AMS_ERR_12
- J10 pad 7: ~{TS_ACT} -> CAN0_L
- J10 pad 8: AMS_ERR_12 -> CAN0_H
- J11 pad 1: CAN1_L -> GND
- J11 pad 2: CAN1_H -> +5V
- J11 pad 3: GND -> CAN1_L
- J11 pad 4: +5V -> CAN1_H
- J6 pad 3: SDC_IN -> ~{AIR-}
- J6 pad 4: ~{PRE} -> SDC_IN
- J6 pad 5: ~{AIR+} -> ~{PRE}
- J6 pad 6: ~{AIR-} -> ~{AIR+}
Routing:
- net +5V: track 214.1 -> 260.8 mm, vias 13 -> 15
- net +12V: track 41.3 -> 81.7 mm, vias 2 -> 4
- net AMS_ERR_12: track 35.8 -> 58.3 mm
- net SDC_IN: track 10.3 -> 28.7 mm
- net SCK: track 43.5 -> 56.3 mm, vias 0 -> 2
- net MISO: track 37.2 -> 49.4 mm, vias 4 -> 5
- net CAN0_H: track 28.9 -> 16.8 mm
- net AMS_ERR: track 38.9 -> 27.8 mm, vias 1 -> 0
- net MOSI: track 38.3 -> 47.7 mm
- net AIR-_5: track 33.1 -> 24.6 mm, vias 0 -> 1
- net ~{AIR-}: track 35.0 -> 43.2 mm
- net PRE_5: track 38.0 -> 31.0 mm, vias 2 -> 1
- net PRE_R_T_input: track 13.7 -> 7.82 mm, vias 1 -> 0
- net CAN0_L: track 24.8 -> 19.1 mm
- net Net-(Q3-B): track 0.00 -> 4.11 mm
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
Commit message: sleepy
Parts:
- moved CA2 54.6 mm to (153.4, 60.5)
- moved CA3 54.6 mm to (144.2, 60.6)
- moved CA4 54.6 mm to (139.6, 60.5)
- moved CA5 54.6 mm to (148.7, 60.6)
- moved D10 54.6 mm to (153.6, 56.3)
- moved D11 54.6 mm to (148.9, 56.3)
- moved D8 54.6 mm to (139.9, 56.3)
- moved D9 54.6 mm to (144.5, 56.3)
- moved R53 54.6 mm to (153.4, 58.5)
- moved R55 54.6 mm to (144.2, 58.5)
- moved R56 54.6 mm to (153.4, 60.5)
- moved R57 54.6 mm to (144.2, 60.6)
- moved R58 54.6 mm to (148.7, 60.6)
- moved R59 54.6 mm to (139.6, 60.5)
- moved R60 54.6 mm to (149.7, 67.4)
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Connections:
- J10 pad 1: SDC_IN -> ~{TS_ACT}
- J10 pad 3: ~{TS_ACT} -> SDC_IN
- J12 pad 3: GND -> +5V
- J12 pad 4: +5V -> GND
- J6 pad 3: ~{AIR-} -> SDC_IN
- J6 pad 4: SDC_IN -> ~{PRE}
- J6 pad 5: ~{PRE} -> ~{AIR+}
- J6 pad 6: ~{AIR+} -> ~{AIR-}
- U12 pad 10: TS_ACT_5 -> CAN1_CS
- U12 pad 11: SDC_5 -> CAN0_CS
- U12 pad 13: CAN0_CS -> SDC_5
- U12 pad 14: CAN1_CS -> TS_ACT_5
Routing:
- net +12V: track 81.7 -> 233.3 mm
- net RST: track 29.1 -> 140.2 mm, vias 3 -> 5
- net +5V: track 260.8 -> 364.9 mm, vias 15 -> 16
- net CAN1_H: track 3.54 -> 48.7 mm
- net CAN1_L: track 3.54 -> 45.5 mm
- net INPUT2: track 4.25 -> 39.5 mm, vias 1 -> 2
- net SDC_IN: track 28.7 -> 60.5 mm, vias 0 -> 1
- net RST_12: track 4.29 -> 32.2 mm, vias 1 -> 3
- net ~{TS_ACT}: track 4.35 -> 29.6 mm, vias 1 -> 2
- net TS_ACT_5: track 39.1 -> 22.4 mm, vias 0 -> 1
- net TS-_T: track 86.7 -> 75.3 mm
- net PRE_R_T: track 89.9 -> 78.9 mm
- net HALL_LO: track 58.6 -> 51.1 mm
- net SDC_5: track 35.3 -> 29.0 mm, vias 0 -> 1
- net PRE_R_T_input: track 7.82 -> 13.2 mm
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
Commit message: hi
Parts:
- J10: footprint Connector_Molex:Molex_Micro-Fit_3.0_43045-0800_2x04_P3.00mm_Horizontal -> RMC_Connnector:Molex_Micro-Fit_3.0_43045-0800_2x04_P3.00mm_Horizontal_BiggerPad
- J11, J12, J13: footprint Connector_Molex:Molex_Micro-Fit_3.0_43045-0400_2x02_P3.00mm_Horizontal -> RMC_Connnector:Molex_Micro-Fit_3.0_43045-0400_2x02_P3.00mm_Horizontal_BiggerPad
- J6: footprint Connector_Molex:Molex_Micro-Fit_3.0_43045-0600_2x03_P3.00mm_Horizontal -> RMC_Connnector:Molex_Micro-Fit_3.0_43045-0600_2x03_P3.00mm_Horizontal_BiggerPad
- J7: footprint Connector_Molex:Molex_Micro-Fit_3.0_43045-0200_2x01_P3.00mm_Horizontal -> RMC_Connnector:Molex_Micro-Fit_3.0_43045-0200_2x01_P3.00mm_Horizontal_BiggerPad
- moved J10 0.60 mm to (170.3, 62.7)
- moved J7 0.50 mm to (127.5, 49.8)
- moved J6 0.30 mm to (170.3, 80.0)
Routing:
- net INPUT2: track 39.5 -> 38.1 mm
- net Net-(U13-OSC1): track 11.1 -> 12.1 mm
- net HALL_HI: track 58.4 -> 59.3 mm
- net ~{TS_ACT}: track 29.6 -> 29.0 mm
- net AMS_ERR_12: track 58.3 -> 58.9 mm
- net GND: vias 35 -> 32

Commit message: BDUCUM
BDUCU changes
Parts:
- CA1: moved to F.Cu
- R54: moved to B.Cu
- moved AVR-ISP1 5.68 mm to (160.3, 69.5), turned to 0 degrees
- moved C15 3.28 mm to (113.2, 70.8), turned to -90 degrees
- moved C12 1.70 mm to (107.8, 78.8)
- moved C14 1.70 mm to (110.8, 78.8)
- moved CA1 1.14 mm to (156.8, 67.6), turned to -90 degrees
Routing:
- net +5V: track 365.3 -> 340.1 mm, vias 16 -> 17
- net GND: track 0.00 -> 15.6 mm, vias 32 -> 117
- net MOSI: track 47.9 -> 52.1 mm
- net RST: track 140.2 -> 137.5 mm
- net AC_ISO: track 21.7 -> 24.3 mm, vias 0 -> 2
- net MISO: track 50.0 -> 49.2 mm, vias 5 -> 4
- net +12V: track 233.4 -> 234.2 mm
- net SCK: track 56.3 -> 56.9 mm

Commit message: update silkscreen
Other:
- board text added: "RBR_AMS_MASTER_V1.1 25/08/2026 PCB by Nicholas Chan"
- board text removed: "RBR_AMS_MASTER_V1.1 22/08/2026 PCB by Nicholas Chan"

Commit message: reviewed Jasmine's BDUCU version
Routing:
- net +5V: track 340.1 -> 337.5 mm
- net HALL_HI: track 59.3 -> 56.8 mm
- net CAN0_H: track 16.9 -> 14.5 mm
- net Net-(U13-OSC1): track 12.1 -> 10.4 mm
- net GND: track 15.6 -> 17.2 mm, vias 117 -> 291
- net PRE_R_T_input: track 13.2 -> 12.5 mm
- net XTAL1: track 10.3 -> 9.81 mm
- net +12V: track 234.2 -> 233.7 mm, vias 4 -> 3
- net CAN0_L: track 19.3 -> 18.8 mm
- net RST_12: track 31.9 -> 31.8 mm, vias 3 -> 2

Commit message: update sorry I draw shit board
Parts:
- removed R64, R65, R66, R67: 4.7k, RMC_Resistor:R_0805_2012Metric_Pad1.20x1.40mm_HandSolder_L
- R21, R22: value 100k -> 10k
- moved CA4 1.02 mm to (138.6, 60.5)
- moved R52 1.02 mm to (138.7, 58.5)
- moved R59 1.02 mm to (138.6, 60.5)
- moved D8 1.02 mm to (138.9, 56.3)
- moved D9 0.67 mm to (143.8, 56.3)
- moved R55 0.67 mm to (143.6, 58.4)
- moved CA3 0.67 mm to (143.6, 60.5)
- moved R57 0.67 mm to (143.6, 60.5)
- moved U10 0.64 mm to (155.0, 79.8)
- moved U13 0.40 mm to (138.1, 79.8)
- moved C26 0.40 mm to (117.6, 89.8)
- moved C27 0.40 mm to (127.3, 89.8)
- moved R28 0.40 mm to (122.5, 89.8)
- moved R54 0.22 mm to (148.5, 58.4)
- moved D11 0.22 mm to (148.7, 56.3)
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Connections:
- J13 pad 3: GND -> +5V
- J13 pad 4: GND -> +5V
- U16 pad 10: TS_ACT_5 -> +5V
- U16 pad 11: GND -> RST
- U16 pad 12: RST -> +5V
- U16 pad 13: GND -> SDC_5
- U16 pad 14: SDC_5 -> +5V
- U16 pad 15: GND -> INPUT2_5V
- U16 pad 16: INPUT2_5V -> +5V
- U16 pad 9: GND -> TS_ACT_5
Routing:
- net +5V: track 337.5 -> 352.1 mm, vias 17 -> 18
- net INPUT2_5V: track 34.6 -> 26.5 mm, vias 1 -> 0
- net SDC_5: track 28.9 -> 24.0 mm, vias 1 -> 0
- net INPUT2: track 38.1 -> 42.7 mm
- net TS_ACT_5: track 22.3 -> 18.2 mm, vias 1 -> 0
- net RST: track 137.3 -> 133.6 mm
- net +12V: track 233.7 -> 236.1 mm
- net CAN0_H: track 14.5 -> 16.4 mm
- net Net-(U17-SW): track 14.1 -> 15.9 mm
- net HALL_HI: track 56.8 -> 55.7 mm
- net Net-(CA4-Pad1): track 14.9 -> 15.9 mm
- net Net-(CA3-Pad1): track 6.45 -> 7.45 mm
- net XTAL2: track 9.69 -> 10.6 mm
- net SCK: track 56.9 -> 57.7 mm
- net /MCU/CAN1/CAN_RX: track 12.2 -> 13.0 mm
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