File: TSAL_G_HVB_V2/TSAL_G_HVB_V2.kicad_pcb (KiCad board)
At the start: 2 copper layers, 100 x 50 mm, 48 parts, among them J1 Conn_01x03_Pin, J2 Conn_01x02_Pin, J3 Conn_01x02_Pin, J4 Conn_01x02_Pin, Q1 2N7002, Q2 MMBT3904, Q3 PMOS, U1 uA7805, U2 74HC86, U3 74AHC04, U4 74LS09, U5 NE555D

Commit message: TSAL G HVB V2 patch
I SHIT DRAW THIS AT WORK
MIGHT BE SHITTER THEN MINI POWER
Other:
- board text added: "GAY MEAN HAPPY"
- board text added: "SYMMETRICAL AWD IS BETTER THEN VTEC"
- board text removed: "SYMMETRICAL AWD"
