File: SSRU_v4.0/SSRU_v4.0.kicad_pcb (KiCad board)
At the start: 2 copper layers, 95 x 78 mm, 71 parts, among them J2 Conn_01x24, J4 AVR-ISP-6, SW1 SW_Push, U1 SGM722, U10 TJA1051T, U2 ATmega328P-A, U3 SGM722, U4 LM2576S-5, U6 MCP2515-xST, U69 SGM722, Y1 16MHz, Y4 20MHz

Commit message: gay
Connections:
- J2 pad 15: AMBIENT_NTC_50k_IN -> STEER_IN
- J2 pad 17: +5V -> GND
- J2 pad 23: GND -> AMBIENT_NTC_50k_IN
- J2 pad 7: STEER_IN -> +5V
Routing:
- net AMBIENT_NTC_50k_IN: track 62.5 -> 77.3 mm
- net STEER_IN: track 32.7 -> 36.9 mm
- net +5V: track 385.8 -> 384.4 mm
- net GND: vias 663 -> 658

Commit message: KOALA
Parts:
- removed R12, R3: 50k, RMC_Resistor:R_0805_2012Metric_Pad1.20x1.40mm_HandSolder_L
- added G***: LOGO, LOGO, F.Cu at (190.2, 112.8)
- added G***: LOGO, LOGO, F.Cu at (163.8, 76.8)
- added G***: LOGO, LOGO, F.Cu at (179.0, 68.0)
- added G***: LOGO, LOGO, F.Cu at (141.2, 84.2)
- added G***: LOGO, LOGO, F.Cu at (153.7, 131.2)
- added G***: LOGO, LOGO, F.Cu at (162.0, 131.4)
- added G***: LOGO, LOGO, F.Cu at (151.0, 78.2)
- moved R6 5.82 mm to (128.9, 105.9)
- moved C9 2.49 mm to (126.4, 106.0)
- moved JP4 0.15 mm to (142.6, 107.0)
- moved C15 0.15 mm to (150.0, 115.0)
- moved U1 0.13 mm to (156.3, 113.2)
Routing:
- net PUMP_NTC_50k_IN: track 26.3 -> 22.4 mm, vias 2 -> 1
- net +5V: track 384.4 -> 386.8 mm, vias 10 -> 9
- net GND: track 0.00 -> 1.00 mm, vias 658 -> 654
Other:
- board text added: "+12V CANH +5V +5V +5V +5V +5V FLOW"
- board text added: "+5V CAN1L SCL POT1 POT2 PNTC STEER GND"
- board text added: "GND GND SDA GND GND GND ANTC GND"
- board text removed: "+12V CANH +5V +5V +5V +5V STEER FLOW"
- board text removed: "+5V CAN1L SCL POT1 POT2 PNTC ANTC GND"
- board text removed: "+5V GND SDA GND GND GND GND GND"

Commit message: helo
Parts:
- added G***: LOGO, LOGO, B.Cu at (122.0, 129.5)
- added G***: LOGO, LOGO, B.Cu at (186.5, 113.5)
- added G***: LOGO, LOGO, B.Cu at (137.1, 74.9)
- added G***: LOGO, LOGO, B.Cu at (167.5, 72.2)
- added G***: LOGO, LOGO, B.Cu at (146.8, 121.5)
- added G***: LOGO, LOGO, B.Cu at (157.7, 98.4)
- added G***: LOGO, LOGO, B.Cu at (117.2, 71.0)
- added R12: 50k, RMC_Resistor:R_0805_2012Metric_Pad1.20x1.40mm_HandSolder_L, F.Cu at (147.5, 115.0)
- added R3: 50k, RMC_Resistor:R_0805_2012Metric_Pad1.20x1.40mm_HandSolder_L, F.Cu at (123.8, 108.4)
