File: steering_sensor_mount_v1.0/steering_sensor_mount_v1.0.kicad_pcb (KiCad board)
At the start: 2 copper layers, 50 x 50 mm, 100 parts, among them J1 Conn_01x03

Commit message: rename project
Parts:
- added G***: LOGO, LOGO, F.Cu at (133.5, 114.0)
- RV1: value R_Potentiometer -> RK097N
Other:
- board text added: "steering sensor mount v1.0 04/08/2026 Jasmine Lee"
- board text removed: "Steering Sensor Mount 03/08/2026 Jasmine Lee"
