File: Charge cart/Charge cart.kicad_sch (KiCad schematic)
At the start: 0 parts

Commit message: charge kart
Parts:
- added D3, D4, D5, D6, D7, D8: LED, symbol Device:LED
- added F1: 10A, symbol Device:Fuse
- added J1: IEC_60320_C14_Receptacle, symbol Connector:IEC_60320_C14_Receptacle
- added J10, J9: Conn_01x03, Connector_Molex:Molex_Micro-Fit_3.0_43650-0315_1x03_P3.00mm_Vertical, symbol Connector_Generic:Conn_01x03
- added J2: 600V PSU AC input, symbol Connector_Generic:Conn_01x03
- added J3: 12V PSU AC input, symbol Connector_Generic:Conn_01x03
- added J4: 600V PSU DC output, symbol Connector_Generic:Conn_01x02
- added J5: 12V PSU DC output, symbol Connector_Generic:Conn_01x02
- added J6: PL00X-301-10M8, symbol Connector_Generic:Conn_01x03
- added J7: PL00Y-301-10M8, symbol Connector_Generic:Conn_01x03
- added J8: Conn_01x23, symbol Connector_Generic:Conn_01x23
- added K1: PNC113BDA, symbol Relay:Relay_SPST-NC
- added K3: EV200 HAANA, Relay_THT:Relay_DPST_Omron_G2RL-2A, symbol Relay:G2RL-2A
- added R1: discharge resistor, symbol Device:R
- added R2: R_Shunt, symbol Device:R_Shunt
- added SW1, SW2: E-stop, symbol Switch:SW_Push
Connections:
- new net: J1.2 (N), J2.3 (Pin_3), J3.3 (Pin_3)
- new net: J1.3 (PE), J2.2 (Pin_2), J3.2 (Pin_2)
- new net: F1.2, SW1.1
- new net: J7.1 (Pin_1), R2.1
- new net: J6.3 (Pin_3), J7.2 (Pin_2)
- new net: J6.2 (Pin_2), SW1.2
- new net: K1.12, R1.1
- new net +12V: D3.2 (A), F1.1, J5.1 (Pin_1), K3.23, SW2.1
- new net AMP_GND: J10.3 (Pin_3)
- new net AMP_SIGNAL: J10.2 (Pin_2)
- new net AMP_VCC: J10.1 (Pin_1)
- new net AMS_ERR: D4.2 (A), J8.3 (Pin_3)
- new net CANH: J8.5 (Pin_5)
- new net CANL: J8.6 (Pin_6)
- new net CAN_SHIELD: J8.7 (Pin_7)
- new net CHARGER_ERR_12V: D7.2 (A)
- new net CHARGING_ENABLE: SW2.2
- new net GND: D4.1 (K), D5.1 (K), D6.1 (K), D7.1 (K), D8.1 (K), J5.2 (Pin_2)
- new net HV_ON: D3.1 (K), K1.A1, K3.A1
- new net HV_PSU_LIVE: J2.1 (Pin_1), K3.14
- new net HV_RELAY_AUX: K3.24
- new net IMD_ERR: D5.2 (A), J8.4 (Pin_4)
- new net LIVE: J1.1 (L), J3.1 (Pin_1), K3.13
- new net SDC_IN: D8.2 (A), J8.2 (Pin_2), K1.A2, K3.A2
- new net SDC_OUT: J7.3 (Pin_3), J8.1 (Pin_1)
- new net TS+: J4.1 (Pin_1), J6.1 (Pin_1), K1.11
- new net TS-: J4.2 (Pin_2), R1.2, R2.4
- new net TSAL_G: D6.2 (A)
- new net VOLT_GND: J9.3 (Pin_3)
- new net VOLT_SIGNAL: J9.2 (Pin_2)
- new net VOLT_VCC: J9.1 (Pin_1)
Other:
- removed sheet PSU (treat as black box)
- note added: "A control"
- note added: "J"
- note added: "MISSING TSAL-G CONNECTIONS IMD GROUNDING POINT (for Main hoop, now on charger"
- note added: "V control"
