File: TS_indicator/TS_indicator.kicad_sch (KiCad schematic)
At the start: 50 parts, among them J1 Conn_01x02_Pin, J2 Conn_01x02_Pin, J3 Conn_01x02_Pin, J4 Conn_01x02_Pin, Q1 AO3401A, Q2 AO3400A, U1 TLV431, U2 PV15-27B12R3, U3 B1212, U7 LTV-817S

Commit message: added TS indicator
Parts:
- F1: footprint Fuse:Fuse_Littelfuse-NANO2-885 -> Fuse:Fuse_Littelfuse-NANO2-462
Changed lines of the file:
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@@
 			)
 		)
-		(property "Footprint" "Fuse:Fuse_Littelfuse-NANO2-885"
+		(property "Footprint" "Fuse:Fuse_Littelfuse-NANO2-462"
 			(at 45.212 82.55 90)
 			(effects
