File: TSALG_ACCUM_V2/TSALG_ACCUM_V2.kicad_sch (KiCad schematic)
At the start: 97 parts, among them J1 Conn_01x02_Pin, J10 Conn_01x02_Pin, J2 Conn_01x02_Pin, J3 Conn_01x03_Pin, J4 Conn_01x02_Pin, J5 Conn_01x02_Pin, J6 Conn_01x02_Pin, J7 Conn_01x03_Pin, J8 Conn_01x02_Pin, J9 Conn_01x03_Pin, U1 TLV431, U10 LM393, U11 LM393, U12 LM393, U2 LTV-817S, U3 B1212, U4 LTV-847S, U5 uA7805, U6 TLV431, U7 MCP6002-xSN, U8 LM393, U9 LM393

Commit message: ACCUM BOARDs BATCH ORDER
ts indicator
imd latch v2
tsalg accum v2.1
tsalg hvb v2.1
batch order
Parts:
- F1: footprint Fuse:Fuse_Littelfuse-NANO2-885 -> Fuse:Fuse_Littelfuse-NANO2-462
Changed lines of the file:
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@@
 			)
 		)
-		(property "Footprint" "Fuse:Fuse_Littelfuse-NANO2-885"
+		(property "Footprint" "Fuse:Fuse_Littelfuse-NANO2-462"
 			(at 34.29 43.942 90)
 			(hide yes)
