File: IMD_AMS_latch/latch_to_low.kicad_sch (KiCad schematic)
At the start: 6 parts

Commit message: IMD AMS latch
Parts:
- removed C?: 100n, Capacitor_SMD:C_0805_2012Metric_Pad1.18x1.45mm_HandSolder, symbol Device:C
- removed U? (x5): 4001, RMC-KiCad:SOIC127P600X175-14N, symbol 4xxx:4001
- added C2: C, Capacitor_SMD:C_0805_2012Metric_Pad1.18x1.45mm_HandSolder, symbol Device:C
- added U1: 4001, RMC-KiCad:SOIC127P600X175-14N, symbol 4xxx:4001
Connections:
- net +12V: now also C2.1, U1.14 (VDD)
- net GND: now also C2.2, U1.7 (VSS)
- net reset: now also U1.6
- net signal_in: now also U1.9
- net signal_out: now also U1.3, U1.5
- new net: U1.1, U1.11
- new net: U1.10, U1.12, U1.13
- new net: U1.2, U1.4, U1.8
