File: IMD_AMS_latch/IMD_AMS_latch.kicad_pcb (KiCad board)
At the start: 2 copper layers, 66.9 x 59.9 mm, 0 parts

Commit message: IMD AMS latch
Parts:
- added C1: C, Capacitor_SMD:C_0805_2012Metric_Pad1.18x1.45mm_HandSolder, F.Cu at (138.6, 100.8)
- added C2: C, Capacitor_SMD:C_0805_2012Metric_Pad1.18x1.45mm_HandSolder, B.Cu at (184.0, 109.2)
- added C3: C, Capacitor_SMD:C_0805_2012Metric_Pad1.18x1.45mm_HandSolder, B.Cu at (157.2, 99.3)
- added C4: 10u, Capacitor_SMD:C_0805_2012Metric_Pad1.18x1.45mm_HandSolder, F.Cu at (172.6, 96.8)
- added C5: 10u, Capacitor_SMD:C_0805_2012Metric_Pad1.18x1.45mm_HandSolder, F.Cu at (169.2, 111.7)
- added C6: C, Capacitor_SMD:C_0805_2012Metric_Pad1.18x1.45mm_HandSolder, B.Cu at (184.0, 104.0)
- added C7: C, Capacitor_SMD:C_0805_2012Metric_Pad1.18x1.45mm_HandSolder, B.Cu at (157.7, 104.3)
- added D1: 1N4148, Diode_THT:D_DO-35_SOD27_P7.62mm_Horizontal, F.Cu at (168.4, 104.5)
- added D2: 1N4148, Diode_THT:D_DO-35_SOD27_P7.62mm_Horizontal, F.Cu at (173.7, 104.1)
- added D3: 1N4148, Diode_THT:D_DO-35_SOD27_P7.62mm_Horizontal, F.Cu at (134.9, 68.8)
- added D4: LED, LED_SMD:LED_0805_2012Metric_Pad1.15x1.40mm_HandSolder, F.Cu at (185.4, 87.2)
- added D5: LED, LED_SMD:LED_0805_2012Metric_Pad1.15x1.40mm_HandSolder, F.Cu at (134.3, 79.7)
- added D6: 1N4148, Diode_THT:D_DO-35_SOD27_P7.62mm_Horizontal, F.Cu at (176.9, 71.6)
- added D7: LED, LED_SMD:LED_0805_2012Metric_Pad1.15x1.40mm_HandSolder, F.Cu at (180.4, 79.9)
- added D8: 1N4148, Diode_SMD:D_0805_2012Metric_Pad1.15x1.40mm_HandSolder, B.Cu at (179.9, 104.2)
- added D9: 1N4148, Diode_SMD:D_0805_2012Metric_Pad1.15x1.40mm_HandSolder, B.Cu at (162.7, 104.2)
- added H1: MountingHole, MountingHole:MountingHole_4.3mm_M4, F.Cu at (135.0, 60.8)
- added H2: MountingHole, MountingHole:MountingHole_4.3mm_M4, F.Cu at (191.5, 60.7)
- added H3: MountingHole, MountingHole:MountingHole_4.3mm_M4, F.Cu at (134.9, 110.6)
- added H4: MountingHole, MountingHole:MountingHole_4.3mm_M4, F.Cu at (191.5, 110.7)
- added J1: Conn_01x03, Connector_PinHeader_2.54mm:PinHeader_1x03_P2.54mm_Vertical, F.Cu at (153.7, 111.4)
- added J10: Conn_01x02, Connector_Molex:Molex_Micro-Fit_3.0_43650-0200_1x02_P3.00mm_Horizontal, F.Cu at (168.8, 62.7)
- added J12: Conn_01x04, Connector_Molex:Molex_Micro-Fit_3.0_43045-0400_2x02_P3.00mm_Horizontal, F.Cu at (157.4, 62.7)
- added J2: Conn_01x03, Connector_PinHeader_2.54mm:PinHeader_1x03_P2.54mm_Vertical, F.Cu at (188.3, 96.6)
- added J3: Conn_01x04, Connector_Molex:Molex_Micro-Fit_3.0_43045-0400_2x02_P3.00mm_Horizontal, F.Cu at (189.0, 81.7)
- added J4: Conn_01x04, Connector_Molex:Molex_Micro-Fit_3.0_43045-0400_2x02_P3.00mm_Horizontal, F.Cu at (189.0, 69.8)
- added J7: Conn_01x02, Connector_Molex:Molex_Micro-Fit_3.0_43650-0215_1x02_P3.00mm_Vertical, F.Cu at (153.7, 89.2)
- added J8: Conn_01x02, Connector_Molex:Molex_Micro-Fit_3.0_43650-0200_1x02_P3.00mm_Horizontal, F.Cu at (145.3, 62.6)
- added J9: Conn_01x02, Connector_Molex:Molex_Micro-Fit_3.0_43650-0200_1x02_P3.00mm_Horizontal, F.Cu at (180.0, 62.7)
- added K1: SANYOU_SRD_Form_C, Relay_THT:Relay_SPDT_SANYOU_SRD_Series_Form_C, F.Cu at (144.7, 66.9)
- added K2: SANYOU_SRD_Form_C, Relay_THT:Relay_SPDT_SANYOU_SRD_Series_Form_C, F.Cu at (171.8, 75.0)
- added Q1: AO3400A, Package_TO_SOT_SMD:SOT-23, B.Cu at (144.1, 74.2)
- added Q2: AO3400A, Package_TO_SOT_SMD:SOT-23, B.Cu at (170.1, 85.4)
- added Q3: AO3400A, Package_TO_SOT_SMD:SOT-23, F.Cu at (145.2, 104.7)
- added Q4: AO3401A, Package_TO_SOT_SMD:SOT-23, F.Cu at (145.2, 108.9)
- added Q5: AO3400A, Package_TO_SOT_SMD:SOT-23, F.Cu at (145.2, 100.8)
- added Q6: AO3401A, Package_TO_SOT_SMD:SOT-23, F.Cu at (145.2, 96.8)
- added R1: 0R, Resistor_SMD:R_0805_2012Metric_Pad1.20x1.40mm_HandSolder, F.Cu at (150.9, 110.6)
- added R10: 1k, Resistor_SMD:R_0805_2012Metric_Pad1.20x1.40mm_HandSolder, B.Cu at (185.9, 87.2)
- added R11: R_US, Resistor_SMD:R_0805_2012Metric_Pad1.20x1.40mm_HandSolder, B.Cu at (175.7, 85.3)
- added R12: 0R, Resistor_SMD:R_0805_2012Metric_Pad1.20x1.40mm_HandSolder, F.Cu at (191.1, 97.4)
- added R13: 0R, Resistor_SMD:R_0805_2012Metric_Pad1.20x1.40mm_HandSolder, F.Cu at (191.1, 101.2)
- added R14: R_US, Resistor_SMD:R_0805_2012Metric_Pad1.20x1.40mm_HandSolder, B.Cu at (177.8, 61.9)
- added R15: R_US, Resistor_SMD:R_0805_2012Metric_Pad1.20x1.40mm_HandSolder, B.Cu at (166.6, 61.7)
- added R16: R_US, Resistor_SMD:R_0805_2012Metric_Pad1.20x1.40mm_HandSolder, F.Cu at (134.2, 84.1)
- added R17: R_US, Resistor_SMD:R_0805_2012Metric_Pad1.20x1.40mm_HandSolder, F.Cu at (180.8, 75.3)
- added R18: 1k, Resistor_SMD:R_0805_2012Metric_Pad1.20x1.40mm_HandSolder, F.Cu at (173.9, 99.9)
- added R19: 1k, Resistor_SMD:R_0805_2012Metric_Pad1.20x1.40mm_HandSolder, F.Cu at (168.2, 108.3)
- added R2: 0R, Resistor_SMD:R_0805_2012Metric_Pad1.20x1.40mm_HandSolder, F.Cu at (150.9, 106.8)
- added R20: 1k, Resistor_SMD:R_0805_2012Metric_Pad1.20x1.40mm_HandSolder, F.Cu at (171.3, 99.8)
- added R21: 1k, Resistor_SMD:R_0805_2012Metric_Pad1.20x1.40mm_HandSolder, F.Cu at (170.4, 108.4)
- added R22: R, Resistor_SMD:R_0805_2012Metric_Pad1.20x1.40mm_HandSolder, F.Cu at (141.2, 100.8)
- added R23: R, Resistor_SMD:R_0805_2012Metric_Pad1.20x1.40mm_HandSolder, F.Cu at (148.0, 104.5)
- added R24: R, Resistor_SMD:R_0805_2012Metric_Pad1.20x1.40mm_HandSolder, F.Cu at (139.8, 97.8)
- added R25: R, Resistor_SMD:R_0805_2012Metric_Pad1.20x1.40mm_HandSolder, F.Cu at (149.0, 101.7)
- added R5: R_US, Resistor_SMD:R_0805_2012Metric_Pad1.20x1.40mm_HandSolder, B.Cu at (138.2, 74.3)
- added R6: R_US, Resistor_SMD:R_0805_2012Metric_Pad1.20x1.40mm_HandSolder, B.Cu at (140.9, 74.3)
- added R7: R_US, Resistor_SMD:R_0805_2012Metric_Pad1.20x1.40mm_HandSolder, B.Cu at (173.4, 85.4)
- added R8: 2.2k, Resistor_SMD:R_0805_2012Metric_Pad1.20x1.40mm_HandSolder, B.Cu at (190.0, 79.2)
- added R9: 2.2k, Resistor_SMD:R_0805_2012Metric_Pad1.20x1.40mm_HandSolder, B.Cu at (190.1, 87.2)
- added U1: 4001, RMC-KiCad:SOIC127P600X175-14N, F.Cu at (181.3, 109.2)
- added U2: 4001, RMC-KiCad:SOIC127P600X175-14N, F.Cu at (160.6, 99.4)
- added U3: 4011, RMC-KiCad:SOIC127P600X175-14N, F.Cu at (181.3, 99.2)
- added U4: 4011, RMC-KiCad:SOIC127P600X175-14N, F.Cu at (160.5, 108.8)
Routing:
- net +12V: track 0.00 -> 269.2 mm, vias 0 -> 6
- net /IMD_latch: track 0.00 -> 94.5 mm, vias 0 -> 1
- net /falling_edge_trigger/signal_in: track 0.00 -> 70.3 mm
- net /IMD_err_sig: track 0.00 -> 64.5 mm
- net /falling_edge_trigger2/signal_in: track 0.00 -> 59.9 mm
- net /IMD_power_on_reset: track 0.00 -> 47.0 mm, vias 0 -> 1
- net /AMS_err_sig: track 0.00 -> 43.3 mm, vias 0 -> 1
- net /AMS_power_on_reset: track 0.00 -> 36.9 mm, vias 0 -> 1
- net /AMS_latch: track 0.00 -> 32.1 mm, vias 0 -> 1
- net GND: track 0.00 -> 31.5 mm, vias 1 -> 106
- net Net-(D3-A): track 0.00 -> 24.8 mm
- net Net-(D6-A): track 0.00 -> 17.9 mm
- net Net-(D2-A): track 0.00 -> 16.6 mm
- net Net-(U1-Pad2): track 0.00 -> 16.0 mm
- net Net-(D1-A): track 0.00 -> 15.9 mm
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- added copper zone on B.Cu, net /SDC_IN
- added copper zone on F.Cu, net /SDC_IN
- added copper zone on B.Cu, net /SDC_OUT
- added copper zone on F.Cu, net /SDC_OUT
- added copper zone on B.Cu, net GND
- added copper zone on F.Cu, net GND
- added copper zone on B.Cu, net Net-(J7-Pin_1)
- added copper zone on F.Cu, net Net-(J7-Pin_1)
- added copper zone on B.Cu, net Net-(J7-Pin_2)
- added copper zone on F.Cu, net Net-(J7-Pin_2)
Other:
- board text added: "AMS_LATCH"
- board text added: "AMS_RST_BTN"
- board text added: "EXT_LED+ OKHS EXT_LED- OMHS"
- board text added: "GND 12V GND 12V"
- board text added: "IMD_LATCH"
- board text added: "IMD_RST_BTN"
- board text added: "R1 - active_high AMS R2 - active_low AMS R12 - active_high IMD R13 - active_low IMD"
- board text added: "SDC_IN"
- board text added: "SDC_OUT"

Commit message: minor fix on IMD AMS latch
Routing:
- net GND: vias 106 -> 110
Changed lines of the file:
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@@
 			(outputformat 1)
 			(mirror no)
-			(drillshape 1)
+			(drillshape 0)
 			(scaleselection 1)
-			(outputdirectory "")
+			(outputdirectory "output/")
 		)
 	)
@@
 	)
 	(via
+		(at 166.92 68.18)
+		(size 0.6)
+		(drill 0.3)
+		(layers "F.Cu" "B.Cu")
+		(free yes)
+		(net 1)
+	)
+	(via
 		(at 166.51 58.3)
 		(size 0.6)
@@
 	)
 	(via
+		(at 164.39 67.84)
+		(size 0.6)
+		(drill 0.3)
+		(layers "F.Cu" "B.Cu")
+		(free yes)
+		(net 1)
+	)
+	(via
 		(at 134.84 71.91)
 		(size 0.6)
@@
 	)
 	(via
+		(at 167.72 66.64)
+		(size 0.6)
+		(drill 0.3)
+		(layers "F.Cu" "B.Cu")
+		(free yes)
+		(net 1)
+	)
+	(via
 		(at 194.01 58.24)
 		(size 0.6)
@@
 		(size 0.6)
 		(drill 0.3)
+		(layers "F.Cu" "B.Cu")
+		(free yes)
+		(net 1)
+	)
+	(via
+		(at 165.36 66.08)
+		(size 0.6)
+		(drill 0.3)

Commit message: updated schematic, use diode instead of mosfet
Parts:
- removed Q3, Q5: AO3400A, Package_TO_SOT_SMD:SOT-23
- removed Q4, Q6: AO3401A, Package_TO_SOT_SMD:SOT-23
- removed R23, R25: R, Resistor_SMD:R_0805_2012Metric_Pad1.20x1.40mm_HandSolder
- added D10: 1N4148, Diode_SMD:D_0805_2012Metric_Pad1.15x1.40mm_HandSolder, F.Cu at (145.6, 103.8)
- added D11: 1N4148, Diode_SMD:D_0805_2012Metric_Pad1.15x1.40mm_HandSolder, F.Cu at (147.2, 99.3)
Routing:
- net /IMD_err_sig: track 64.5 -> 27.4 mm
- net +12V: track 269.2 -> 245.1 mm, vias 6 -> 5
- net /AMS_err_sig: track 43.3 -> 27.2 mm, vias 1 -> 0
- net GND: track 31.5 -> 26.1 mm, vias 110 -> 114
- net /AMS_power_on_reset: track 36.9 -> 31.7 mm
- net Net-(Q3-D): track 4.17 -> 0.00 mm
- net Net-(Q5-D): track 4.02 -> 0.00 mm
- net Net-(D10-A): track 9.69 -> 10.8 mm
